File: PCB/_autosave-MPU_MOD.kicad_sch (KiCad schematic)
At the start: 1 part, among them U2 STM32MP157FABx

Commit message: pcb update
Parts:
- added C1, C2, C3, C4, C5, C6, C7: 4.7uF, Capacitor_SMD:C_0402_1005Metric, symbol Device:C
- added U1: STPMIC1APQR, STPMIC1APQR:QFN40P600X500X80-45N, symbol STPMIC1APQR:STPMIC1APQR
- added unit 1 of U2
Connections:
- new net: C3.1, U1.18 (LDO2OUT)
- new net: C5.1, U1.20 (LDO5OUT)
- new net: C4.1, U1.39 (LDO4OUT)
- new net: C7.1, U1.40 (INTLDO)
- new net: C6.1, U1.21 (LDO6OUT)
- new net: C2.1, U1.23 (LDO1OUT)
- new net GNDA: C7.2, U1.41 (AGND)
Other:
- removed sheet PWR_MPU
- note added: "CVIN, CLDO1OUT, CLDO2OUT, CLDO4OUT, CLDO5OUT, CLDO6OUT, CINTLDO"

Commit message: PCB_UPDATE
Parts:
- removed unit 1 of U2
Other:
- added sheet MPU_PWR (MPU_PWR.kicad_sch)
