File: PCB/MPU_MOD.kicad_sch (KiCad schematic)
At the start: 2 parts, among them U1 STPMIC1APQR, U2 STM32MP157FABx

Commit message: PCB UPDATE
Parts:
- removed U1: STPMIC1APQR, STPMIC1APQR:QFN40P600X500X80-45N, symbol STPMIC1APQR:STPMIC1APQR
- removed unit 1 of U2
Other:
- added sheet MPU_PWR (MPU_PWR.kicad_sch)
- added sheet PWR (PWR.kicad_sch)

Commit message: PCB_UPDATE. PWR DONE, DDR STARTED
Parts:
- removed unit 2 of U2
Other:
- added sheet DDR (DDR.kicad_sch)
