File: PCB/MPU_MOD.kicad_sch (KiCad schematic)
At the start: 1 part, among them U2 STM32MP157FABx

Commit message: PCB_UPDATE
Parts:
- removed U2: STM32MP157FABx, Package_BGA:ST_LFBGA-354_16x16mm_Layout19x19_P0.8mm, symbol New_Library:STM32MP157FABx
Other:
- added sheet HS_intrf (HS_intrf.kicad_sch)

Commit message: PCB_UPDATE
Other:
- added sheet DAC (DAC.kicad_sch)
- added sheet WIFI_BLE (WIFI_BLE.kicad_sch)
Changed lines of the file:
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@@
+	)
+	(sheet
+		(at 254 161.29)
+		(size 52.07 30.48)
+		(exclude_from_sim no)
+		(in_bom yes)
+		(on_board yes)
+		(dnp no)
+		(fields_autoplaced yes)
+		(stroke
+			(width 0.1524)
+			(type solid)
+		)
+		(fill
+			(color 0 0 0 0.0000)
+		)
+		(property "Sheetname" "WIFI_BLE"
+			(at 254 160.5784 0)
+			(effects
+				(font
+					(size 1.27 1.27)
+				)
+				(justify left bottom)
+			)
+		)
+		(property "Sheetfile" "WIFI_BLE.kicad_sch"
+			(at 254 192.3546 0)
+			(effects
+				(font
+					(size 1.27 1.27)
+				)
+				(justify left top)
+			)
+		)
+		(instances
+			(project "MPU_MOD"
+				(path "/65890f61-d586-475b-928a-b635a5e4e59e"
+					(page "9")
+				)
+			)
+		)
 	)
 	(sheet
@@
 				)
 			)
+		)
+	)
+	(sheet
+		(at 254 204.47)
+		(size 53.34 33.02)
+		(exclude_from_sim no)
+		(in_bom yes)
+		(on_board yes)
+		(dnp no)
+		(fields_autoplaced yes)
+		(stroke
+			(width 0.1524)
+			(type solid)
+		)
+		(fill
+			(color 0 0 0 0.0000)
+		)
+		(property "Sheetname" "DAC"
+			(at 254 203.7584 0)
+			(effects
+				(font
+					(size 1.27 1.27)
+				)
+				(justify left bottom)
+			)
+		)
+		(property "Sheetfile" "DAC.kicad_sch"
+			(at 254 238.0746 0)
+			(effects
+				(font
+					(size 1.27 1.27)
+				)
+				(justify left top)
+			)
+		)
+		(instances
+			(project "MPU_MOD"
+				(path "/65890f61-d586-475b-928a-b635a5e4e59e"
+					(page "10")
+				)
+			)
