File: PCB/PWR.kicad_sch (KiCad schematic)
At the start: 27 parts, among them U1 STPMIC1APQR, U9 STC3115IQT

Commit message: PCB_UPDATE
Parts:
- added BT1: Battery_Cell, symbol Device:Battery_Cell
- added C100, C101, C104, C107, C98, C99: 10uF, Capacitor_SMD:C_0603_1608Metric, symbol Device:C
- added C102: 4.7uF, Capacitor_SMD:C_0402_1005Metric, symbol Device:C
- added C103: 47nF, Capacitor_SMD:C_0402_1005Metric, symbol Device:C
- added C105: 100pF, Capacitor_SMD:C_0402_1005Metric, symbol Device:C
- added C106: 100nF, Capacitor_SMD:C_0402_1005Metric, symbol Device:C
- added C96: 1uF, Capacitor_SMD:C_0402_1005Metric, symbol Device:C
- added C97: 220nF, Capacitor_SMD:C_0402_1005Metric, symbol Device:C
- added D4: LED_B, LED_SMD:LED_0402_1005Metric, symbol Device:LED
- added D5: LED_R, LED_SMD:LED_0402_1005Metric, symbol Device:LED
- added D6: SMAJ5.0A, Diode_SMD:D_SMA, symbol Diode:SMAJ5.0A
- added J3: USB4215-03-A_REVA, USB4215-03-A_REVA:GCT_USB4215-03-A_REVA, symbol USB4215-03-A_REVA:USB4215-03-A_REVA
- added JP4: SolderJumper_3_Bridged12, Jumper:SolderJumper-3_P1.3mm_Bridged12_Pad1.0x1.5mm, symbol Jumper:SolderJumper_3_Bridged12
- added L6: 1uH, Inductor_SMD:L_1008_2520Metric, symbol Device:L
- added R45: 10m, Resistor_SMD:R_0603_1608Metric, symbol Device:R
- added R46, R47: 1k, symbol Device:R
- added R48, R49: 2k2, symbol Device:R
- added R50: 220, symbol Device:R
- added R51: 10k, symbol Device:R
- added R52: 5k23, symbol Device:R
- added R53: 30k1, symbol Device:R
- added R54: 240, symbol Device:R
- added TP16, TP17, TP18, TP19, TP20, TP21: TestPoint, TestPoint:TestPoint_Pad_D1.0mm, symbol Connector:TestPoint
- added U10: BQ25606RGER, BQ25606RGER:QFN50P400X400X100-25N, symbol BQ25606RGER:BQ25606RGER
- added U11: HSP051-4M10, HSP051-4M10:IC_HSP051-4M10, symbol HSP051-4M10:HSP051-4M10
Connections:
- net GND: now also U1.45 (EPGND), U9.5 (GND), C100.1, C101.1, C102.1, C104.1, C105.2, C106.1, C107.1, C96.1, C97.2, C98.1, C99.1, D6.2 (A2), J3.A1_B12 (GND_A), J3.B1_A12 (GND_B), J3.SH1 (SHIELD), J3.SH2 (SHIELD), J3.SH3 (SHIELD), J3.SH4 (SHIELD), JP4.1 (A), R45.2, R46.2, R50.1, R51.1, R53.1, R54.1, U10.17 (GND), U10.18 (GND), U11.3 (GND), U11.8 (GND)
- net at U9.10 (VIN): now also C97.1, R47.1
- net at U9.6 (CG): now also BT1.2 (-), R45.1
- net at U9.8 (BATD/CD): now also R46.1
- net +BATT: now reaches U9.9 (VCC)
- net +BATT: now also BT1.1 (+), C104.2, C96.2, R47.2, U10.13 (BAT), U10.14 (BAT)
- net 5V_VIN renamed VIN
- net VIN: now also C98.2, D4.2 (A), D5.2 (A), L6.2, U10.15 (SYS), U10.16 (SYS)
- new net: D5.1 (K), R49.1, TP17.1
- new net: R50.2, U10.10 (ICHG)
- new net: C103.1, L6.1, U10.19 (SW), U10.20 (SW)
- new net: JP4.2 (C), U10.9 (~{CE})
- new net: R49.2, U10.5 (STAT)
- new net: C103.2, U10.21 (BTST)
- new net: R51.2, U10.12 (VSET)
- new net: D4.1 (K), R48.1, TP16.1
- new net: R48.2, U10.7 (~{PG})
- new net: R54.2, U10.8 (ILIM)
- new net: C99.2, U10.23 (PMID)
- new net BATT_T: R52.1, R53.2, U10.11 (TS)
- new net BAT_CHRG: JP4.3 (B)
- new net OTG_ON: U10.6 (OTG)
- new net REGN: C102.2, R52.2, U10.22 (REGN)
- new net USB_CC1: J3.A5 (CC1), TP21.1, U11.5 (I/O_4), U11.6 (NC)
- new net USB_CC2: J3.B5 (CC2), TP20.1, U11.4 (I/O_3), U11.7 (NC)
- new net USB_D+: J3.A6 (DP1), J3.B6 (DP2), TP19.1, U10.3 (D+), U11.2 (I/O_2), U11.9 (NC)
- new net USB_D-: J3.A7 (DN1), J3.B7 (DN2), TP18.1, U10.4 (D-), U11.1 (I/O_1), U11.10 (NC)
- new net V_USB: C100.2, C101.2, C105.1, C106.2, C107.2, D6.1 (A1), J3.A4_B9 (VBUS_A), J3.B4_A9 (VBUS_B), U10.1 (VAC), U10.24 (VBUS)
Other:
- moved on the sheet: U9

Commit message: PCB_UPDATE
Parts:
- removed C105: 100pF, Capacitor_SMD:C_0402_1005Metric, symbol Device:C
- removed C106: 100nF, Capacitor_SMD:C_0402_1005Metric, symbol Device:C
- removed C107: 10uF, Capacitor_SMD:C_0603_1608Metric, symbol Device:C
- removed D6: SMAJ5.0A, Diode_SMD:D_SMA, symbol Diode:SMAJ5.0A
- removed J3: USB4215-03-A_REVA, USB4215-03-A_REVA:GCT_USB4215-03-A_REVA, symbol USB4215-03-A_REVA:USB4215-03-A_REVA
- removed TP18, TP19, TP20, TP21: TestPoint, TestPoint:TestPoint_Pad_D1.0mm, symbol Connector:TestPoint
- removed U11: HSP051-4M10, HSP051-4M10:IC_HSP051-4M10, symbol HSP051-4M10:HSP051-4M10
- added C113: 10nF, Capacitor_SMD:C_0402_1005Metric, symbol Device:C
- added D7: PTVS3V3S1UR, PTVS3V3S1UR:TVS_PTVS3V3S1UR, symbol PTVS3V3S1UR:PTVS3V3S1UR
- added R58, R59: 10k, Resistor_SMD:R_0402_1005Metric, symbol Device:R
- added S3: PTS525SM15SMTR2LFS, lib:SW_PTS525SM15SMTR2LFS, symbol PTS525SM15SMTR2LFS:PTS525SM15SMTR2LFS
- added TH1: Thermistor, symbol Device:Thermistor
- added TP22, TP23, TP24, TP25, TP26, TP27, TP28, TP29, TP30, TP31: TestPoint, TestPoint:TestPoint_Pad_D1.0mm, symbol Connector:TestPoint
- R40, R46, R47, R48, R49, R50, R51, R52, R53, R54: footprint (none) -> Resistor_SMD:R_0402_1005Metric
- U1: footprint STPMIC1APQR:QFN40P600X500X80-45N -> lib:QFN40P600X500X80-45N
- U10: footprint BQ25606RGER:QFN50P400X400X100-25N -> lib:QFN50P400X400X100-25N
- U9: footprint STC3115IQT:SON50P300X200X60-10N -> lib:SON50P300X200X60-10N
Connections:
- net +BATT: now also R58.2, R59.2, TP31.1
- net 3V3: now also TP25.1
- net BATT_T: now also TH1.1
- net GND: now also C113.1, D7.A, S3.1, S3.2, TH1.2
- net VDD: now also U1.42 (VIO), TP24.1
- net VDDA: now also TP29.1
- net VDD_CORE: now also TP22.1
- net VDD_DDR: now also TP23.1
- net VDD_USB: now also TP28.1
- net VIN: now also TP30.1
- net VREF_DDR: now also TP26.1
- net VTT_DDR: now also TP27.1
- net at U1.17 (~{PONKEY}): now also C113.2, D7.C, S3.3, S3.4
- net PMIC_WAKEUP: now reaches U1.2 (WAKEUP)
- net SYS_I2C_SDA: now reaches U1.3 (SDA)
- net SYS_I2C_SDA: now also U9.3 (SCL)
- net SYS_I2C_SCL: now reaches U1.4 (SCL)
- net SYS_I2C_SCL: now also U9.2 (SDA)
- net PMIC_PA0_WKUP_INTR: now reaches U1.43 (~{INT})
- net CHRG_STAT: now reaches D5.1 (K), R49.1, TP17.1
- net CHRG_NPG: now reaches D4.1 (K), R48.1, TP16.1
- net BAT_FUEL_ALARM: now reaches U9.1 (ALM)
- net BAT_FUEL_ALARM: now also R59.1
- net BAT_FUEL_RSDTIO: now reaches U9.7 (RSTIO)
- net BAT_FUEL_RSDTIO: now also R58.1
- net BAT_CHRG renamed CHRG_OFF
- net OTG_ON renamed CHRG_OTG_ON
