File: PCB/PWR.kicad_sch (KiCad schematic)
At the start: 70 parts, among them U1 STPMIC1APQR, U10 BQ25606RGER, U9 STC3115IQT

Commit message: wifi done
Parts:
- removed JP4: SolderJumper_3_Bridged12, Jumper:SolderJumper-3_P1.3mm_Bridged12_Pad1.0x1.5mm, symbol Jumper:SolderJumper_3_Bridged12
- added R90, R91: 0, Resistor_SMD:R_0402_1005Metric, symbol Device:R
Connections:
- net CHRG_OFF: now also R90.2
- net GND: now also R91.1
- net at U10.9 (~{CE}): now also R90.1, R91.2

Commit message: PCB_UPDATE
Parts:
- removed S3: PTS525SM15SMTR2LFS, lib:SW_PTS525SM15SMTR2LFS, symbol PTS525SM15SMTR2LFS:PTS525SM15SMTR2LFS
- added S201: EVQ-9P701P, lib:SW_EVQ-9P701P, symbol EVQ-9P701P:EVQ-9P701P
- BT201: renamed from BT1; footprint (none) -> Connector_PinHeader_1.00mm:PinHeader_1x02_P1.00mm_Vertical
- D203: renamed from D7; footprint PTVS3V3S1UR:TVS_PTVS3V3S1UR -> lib:TVS_PTVS3V3S1UR
- TH201: renamed from TH1; footprint (none) -> Connector_PinHeader_1.00mm:PinHeader_1x02_P1.00mm_Vertical
- renumbered C101 to C201, C100 to C202, C99 to C203, C97 to C204, C96 to C205, C103 to C206, C102 to C207, C98 to C208, C104 to C209, C113 to C210, C10 to C211, C11 to C212, C12 to C213, C13 to C214, C17 to C215, C8 to C216, C9 to C217, C14 to C218, C16 to C219, C3 to C220, C2 to C221, C15 to C222, C4 to C223, C5 to C224, C6 to C225, C7 to C226, C23 to C227, C22 to C228, C21 to C229, C20 to C230, D5 to D201, D4 to D202, L6 to L201, L1 to L202, L2 to L203, L3 to L204, L4 to L205, R58 to R201, R59 to R202, R90 to R203, R48 to R204, R49 to R205, R50 to R206, R91 to R207, R51 to R208, R46 to R209, R47 to R210, R54 to R211, R45 to R212, R52 to R213, R53 to R214, R40 to R215, TP16 to TP201, TP17 to TP202, TP31 to TP203, TP30 to TP204, TP26 to TP205, TP27 to TP206, TP28 to TP207, TP29 to TP208, TP22 to TP209, TP23 to TP210, TP24 to TP211, TP25 to TP212, U9 to U201, U10 to U202, U1 to U203
Connections:
- net GND: now also S201.2A, S201.2B, S201.2C, S201.2D
- net PWR_SW_WAKE_UP: now reaches C210.2, D203.C, U203.17 (~{PONKEY})
- net PWR_SW_WAKE_UP: now also S201.1A, S201.1B
