File: PCB/DDR.kicad_sch (KiCad schematic)
At the start: 8 parts, among them U2 STM32MP157FABx, U3 MT41K256M16TW-107_P

Commit message: DDR_DONE
Parts:
- added C62, C63, C64, C65, C66, C67, C68, C69, C70, C71, C72, C73, C74, C75, C76, C77, C78, C79, C80, C81, C82, C83, C84, C89: 100nF, Capacitor_SMD:C_0402_1005Metric, symbol Device:C
- added C85, C86: 1uF, Capacitor_SMD:C_0402_1005Metric, symbol Device:C
- added C87, C88: 10uF, Capacitor_SMD:C_0603_1608Metric, symbol Device:C
- added R10, R11, R12, R13, R14, R15, R16, R17, R18, R19, R20, R21, R22, R23, R24, R25, R26, R27, R28, R5, R6, R7, R8, R9: 56, symbol Device:R
- added R29: 240, symbol Device:R
- added TP1, TP2, TP3: TestPoint, TestPoint:TestPoint_Pad_D1.0mm, symbol Connector:TestPoint
Connections:
- net DDR_DML is gone; now on net DDR_DQM1: U3.E7 (LDM)
- net DDR_DMU is gone; now on net DDR_DQM0: U3.D3 (UDM)
- net DDR_A0: now also U2.H18 (DDR_A0), R5.1
- net DDR_A1: now also U2.M17 (DDR_A1), R6.1
- net DDR_A10: now also U2.M19 (DDR_A10), R15.1
- net DDR_A11: now also U2.M18 (DDR_A11), R16.1
- net DDR_A12: now also U2.L17 (DDR_A12), R17.1
- net DDR_A13: now also U2.F17 (DDR_A13), R18.1
- net DDR_A14: now also U2.N18 (DDR_A14), R19.1
- net DDR_A2: now also U2.G18 (DDR_A2), R7.1
- net DDR_A3: now also U2.F19 (DDR_A3), R8.1
- net DDR_A4: now also U2.P17 (DDR_A4), R9.1
- net DDR_A5: now also U2.H17 (DDR_A5), R10.1
- net DDR_A6: now also U2.N16 (DDR_A6), R11.1
- net DDR_A7: now also U2.E17 (DDR_A7), R12.1
- net DDR_A8: now also U2.R17 (DDR_A8), R13.1
- net DDR_A9: now also U2.G17 (DDR_A9), R14.1
- net DDR_BA0: now also U2.G19 (DDR_BA0), R20.1
- net DDR_BA1: now also U2.N17 (DDR_BA1), R21.1
- net DDR_BA2: now also U2.J16 (DDR_BA2), R22.1
- net DDR_CASN: now also U2.K17 (DDR_CASN), R26.1
- net DDR_CKE: now also U2.P19 (DDR_CKE), R25.1
- net DDR_CLK_N: now also U2.K19 (DDR_CLKN)
- net DDR_CLK_P: now also U2.L19 (DDR_CLKP)
- net DDR_CSN: now also U2.J18 (DDR_CSN), R24.1
- net DDR_DQ0: now also U2.A17 (DDR_DQ0)
- net DDR_DQ1: now also U2.A18 (DDR_DQ1)
- net DDR_DQ10: now also U2.R18 (DDR_DQ10)
- net DDR_DQ11: now also U2.V19 (DDR_DQ11)
- net DDR_DQ12: now also U2.W18 (DDR_DQ12)
- net DDR_DQ13: now also U2.T18 (DDR_DQ13)
- net DDR_DQ14: now also U2.V18 (DDR_DQ14)
- net DDR_DQ15: now also U2.W17 (DDR_DQ15)
- net DDR_DQ2: now also U2.D18 (DDR_DQ2)
- net DDR_DQ3: now also U2.B17 (DDR_DQ3)
- net DDR_DQ4: now also U2.E18 (DDR_DQ4)
- net DDR_DQ5: now also U2.D17 (DDR_DQ5)
- net DDR_DQ6: now also U2.D19 (DDR_DQ6)
- net DDR_DQ7: now also U2.B18 (DDR_DQ7)
- net DDR_DQ8: now also U2.P18 (DDR_DQ8)
- net DDR_DQ9: now also U2.T17 (DDR_DQ9)
- net DDR_DQS0_N: now also U2.B19 (DDR_DQS0N)
- net DDR_DQS0_P: now also U2.C19 (DDR_DQS0P)
- net DDR_DQS1_N: now also U2.T19 (DDR_DQS1N)
- net DDR_DQS1_P: now also U2.U19 (DDR_DQS1P)
- net DDR_ODT: now also U2.H19 (DDR_ODT), R23.1
- net DDR_RASN: now also U2.L18 (DDR_RASN), R27.1
- net DDR_RESETN: now also U2.G16 (DDR_RESETN)
- net DDR_WEN: now also U2.J17 (DDR_WEN), R28.1
- net GND: now also C62.2, C63.2, C64.2, C65.2, C66.2, C67.2, C68.2, C69.2, C70.2, C71.2, C72.2, C73.2, C74.1, C75.1, C76.1, C77.1, C78.1, C79.1, C80.1, C81.1, C82.1, C83.1, C84.1, C85.2, C86.2, C87.1, C88.1, C89.1, R29.2
- net VDD_DDR: now also C74.2, C75.2, C76.2, C77.2, C78.2, C79.2, C80.2, C81.2, C82.2, C83.2, C84.2, C85.1, C86.1, C87.2, C88.2
- net VREF_DDR: now also U2.W16 (DDR_VREF), C89.2
- net DDR_DQM0: now reaches U2.C18 (DDR_DQM0)
- net at U2.F18 (DDR_ZQ): now also R29.1
- net at U2.J19 (DDR_DTO1): now also TP2.1
- net at U2.K18 (DDR_DTO0): now also TP3.1
- net at U2.N19 (DDR_ATO): now also TP1.1
- net DDR_DQM1: now reaches U2.U18 (DDR_DQM1)
- new net VTT_DDR: C62.1, C63.1, C64.1, C65.1, C66.1, C67.1, C68.1, C69.1, C70.1, C71.1, C72.1, C73.1, R10.2, R11.2, R12.2, R13.2, R14.2, R15.2, R16.2, R17.2, R18.2, R19.2, R20.2, R21.2, R22.2, R23.2, R24.2, R25.2, R26.2, R27.2, R28.2, R5.2, R6.2, R7.2, R8.2, R9.2
- no-connect marks 0 -> 1
Other:
- moved on the sheet: C60, C61, R1, R2, R3, R4, U3

Commit message: PCB_UPDATE
Parts:
- R1, R10, R11, R12, R13, R14, R15, R16, R17, R18, R19, R2, R20, R21, R22, R23, R24, R25, R26, R27, R28, R29, R3, R4, R5, R6, R7, R8, R9: footprint (none) -> Resistor_SMD:R_0402_1005Metric
- U3: footprint MT41K256M16TW-107_P:BGA96C80P9X16_1400X800X120 -> lib:BGA96C80P9X16_1400X800X120

Commit message: PCB_UPDATE
Parts:
- renumbered C89 to C401, C60 to C402, C61 to C403, C85 to C404, C84 to C405, C76 to C406, C62 to C407, C63 to C408, C64 to C409, C65 to C410, C66 to C411, C67 to C412, C68 to C413, C69 to C414, C70 to C415, C71 to C416, C72 to C417, C73 to C418, C86 to C419, C83 to C420, C77 to C421, C87 to C422, C82 to C423, C78 to C424, C88 to C425, C74 to C426, C79 to C427, C75 to C428, C80 to C429, C81 to C430, R29 to R401, R1 to R402, R2 to R403, R3 to R404, R4 to R405, R5 to R406, R6 to R407, R7 to R408, R8 to R409, R9 to R410, R10 to R411, R11 to R412, R12 to R413, R13 to R414, R14 to R415, R15 to R416, R16 to R417, R17 to R418, R18 to R419, R19 to R420, R20 to R421, R21 to R422, R22 to R423, R23 to R424, R24 to R425, R25 to R426, R26 to R427, R27 to R428, R28 to R429, TP1 to TP401, TP2 to TP402, TP3 to TP403, U2 to U301, U3 to U401

Commit message: PCB_UPDATE
Connections:
- net DDR_DQ10: now also U401.C2 (DQ11); no longer U401.C8 (DQ10)
- net DDR_DQ11: now also U401.D7 (DQ8); no longer U401.C2 (DQ11)
- net DDR_DQ12: now also U401.B8 (DQ14); no longer U401.A7 (DQ12)
- net DDR_DQ14: now also U401.C8 (DQ10); no longer U401.B8 (DQ14)
- net DDR_DQ15: now also U401.A7 (DQ12); no longer U401.A3 (DQ15)
- net DDR_DQ8: now also U401.A3 (DQ15); no longer U401.D7 (DQ8)
