File: PCB/DDR.kicad_sch (KiCad schematic)
At the start: 64 parts, among them U301 STM32MP157FABx, U401 MT41K256M16TW-107_P

Commit message: PCB_UPDATE
Connections:
- net DDR_DQ0: now also U401.A2 (DQ13); no longer U401.E3 (DQ0)
- net DDR_DQ1: now also U401.C3 (DQ9); no longer U401.F7 (DQ1)
- net DDR_DQ10: now also U401.G2 (DQ6); no longer U401.C2 (DQ11)
- net DDR_DQ11: now also U401.H8 (DQ5); no longer U401.D7 (DQ8)
- net DDR_DQ12: now also U401.F7 (DQ1); no longer U401.B8 (DQ14)
- net DDR_DQ13: now also U401.H3 (DQ4); no longer U401.A2 (DQ13)
- net DDR_DQ14: now also U401.H7 (DQ7); no longer U401.C8 (DQ10)
- net DDR_DQ15: now also U401.F8 (DQ3); no longer U401.A7 (DQ12)
- net DDR_DQ2: now also U401.A7 (DQ12); no longer U401.F2 (DQ2)
- net DDR_DQ3: now also U401.C2 (DQ11); no longer U401.F8 (DQ3)
- net DDR_DQ4: now also U401.B8 (DQ14); no longer U401.H3 (DQ4)
- net DDR_DQ5: now also U401.C8 (DQ10); no longer U401.H8 (DQ5)
- net DDR_DQ6: now also U401.D7 (DQ8); no longer U401.G2 (DQ6)
- net DDR_DQ7: now also U401.A3 (DQ15); no longer U401.H7 (DQ7)
- net DDR_DQ8: now also U401.F2 (DQ2); no longer U401.A3 (DQ15)
- net DDR_DQ9: now also U401.E3 (DQ0); no longer U401.C3 (DQ9)

Commit message: PCB_UPDATE
Connections:
- net DDR_DQ4: now also U401.C8 (DQ10); no longer U401.B8 (DQ14)
- net DDR_DQ5: now also U401.B8 (DQ14); no longer U401.C8 (DQ10)
Changed lines of the file:
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@@
 	(wire
 		(pts
+			(xy 266.7 162.56) (xy 292.1 162.56)
+		)
+		(stroke
+			(width 0)
+			(type default)
+		)
+	)
+	(wire
+		(pts
 			(xy 323.85 73.66) (xy 326.39 73.66)
 		)
@@
 	(wire
 		(pts
-			(xy 266.7 162.56) (xy 292.1 162.56)
-		)
-		(stroke
-			(width 0)
-			(type default)
-		)
-	)
-	(wire
-		(pts
 			(xy 318.77 107.95) (xy 323.85 107.95)
 		)
@@
 	(wire
 		(pts
-			(xy 266.7 152.4) (xy 292.1 152.4)
-		)
-		(stroke
-			(width 0)
-			(type default)
-		)
-	)
-	(wire
-		(pts
 			(xy 318.77 127) (xy 323.85 127)
 		)
@@
 	(wire
 		(pts
+			(xy 266.7 152.4) (xy 292.1 152.4)
+		)
+		(stroke
+			(width 0)
+			(type default)
+		)
+	)
+	(wire
+		(pts
 			(xy 336.55 130.81) (xy 336.55 133.35)
 		)
@@
 	)
 	(label "DDR_DQ4"
-		(at 292.1 162.56 180)
+		(at 292.1 152.4 180)
 		(effects
 			(font
@@
 	)
 	(label "DDR_DQ5"
-		(at 292.1 152.4 180)
+		(at 292.1 162.56 180)
 		(effects
 			(font

Commit message: pcb_update
Parts:
- added R430: 56, Resistor_SMD:R_0402_1005Metric, symbol Device:R
- added U1: MT41K256M16TW-107_P, MT41K256M16TW-107_P:BGA96C80P9X16_1400X800X120, symbol MT41K256M16TW-107_P_test:MT41K256M16TW-107_P
- U401: footprint lib:BGA96C80P9X16_1400X800X120 -> MT41K256M16TW-107_P:BGA96C80P9X16_1400X800X120; MAXIMUM_PACKAGE_HEIGHT (none) -> 1.20mm; PARTREV (none) -> P; STANDARD (none) -> IPC-7351B
Connections:
- net VTT_DDR: now also R430.2
- net DDR_A15: now reaches U401.M7 (A15)
- net DDR_A15: now also U301.L16 (DDR_A15), R430.1
- new net: U1.A1 (VDDQ), U1.A8 (VDDQ), U1.C1 (VDDQ), U1.C9 (VDDQ), U1.D2 (VDDQ), U1.E9 (VDDQ), U1.F1 (VDDQ), U1.H2 (VDDQ), U1.H9 (VDDQ)
- new net: U1.A9 (VSS), U1.B3 (VSS), U1.E1 (VSS), U1.G8 (VSS), U1.J2 (VSS), U1.J8 (VSS), U1.M1 (VSS), U1.M9 (VSS), U1.P1 (VSS), U1.P9 (VSS), U1.T1 (VSS), U1.T9 (VSS)
- new net: U1.B1 (VSSQ), U1.B9 (VSSQ), U1.D1 (VSSQ), U1.D8 (VSSQ), U1.E2 (VSSQ), U1.E8 (VSSQ), U1.F9 (VSSQ), U1.G1 (VSSQ), U1.G9 (VSSQ)
- new net: U1.B2 (VDD), U1.D9 (VDD), U1.G7 (VDD), U1.K2 (VDD), U1.K8 (VDD), U1.N1 (VDD), U1.N9 (VDD), U1.R1 (VDD), U1.R9 (VDD)
- new net: U1.J1 (NC), U1.J9 (NC), U1.L1 (NC), U1.L9 (NC), U1.M7 (NC)
- no-connect marks 1 -> 0
Other:
- moved on the sheet: R421, R422, R423

Commit message: PCB_UPDATE
Parts:
- removed U1: MT41K256M16TW-107_P, MT41K256M16TW-107_P:BGA96C80P9X16_1400X800X120, symbol MT41K256M16TW-107_P_test:MT41K256M16TW-107_P
- U401: footprint MT41K256M16TW-107_P:BGA96C80P9X16_1400X800X120 -> lib:BGA96C80P9X16_1400X800X120

Commit message: PCB_UPDATE
Parts:
- TP401, TP402, TP403: footprint TestPoint:TestPoint_Pad_D1.0mm -> Library:TP_0.5mm
Changed lines of the file:
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@@
 			)
 		)
-		(property "Footprint" "TestPoint:TestPoint_Pad_D1.0mm"
+		(property "Footprint" "Library:TP_0.5mm"
 			(at 168.91 148.59 0)
 			(effects
@@
 			)
 		)
-		(property "Footprint" "TestPoint:TestPoint_Pad_D1.0mm"
+		(property "Footprint" "Library:TP_0.5mm"
 			(at 162.56 148.59 0)
 			(effects
@@
 			)
 		)
-		(property "Footprint" "TestPoint:TestPoint_Pad_D1.0mm"
+		(property "Footprint" "Library:TP_0.5mm"
 			(at 156.21 148.59 0)
 			(effects
