File: PCB/MPU_MOD.kicad_pcb (KiCad board)
At the start: 2 copper layers, 26 parts, among them U2 STM32MP157FABx

Commit message: PCB_UPDATE
Parts:
- added C1: CPH3225A, lib:CAPCP3225X100N, F.Cu at (176.3, 111.0)
- added C100: 10uF, Capacitor_SMD:C_0603_1608Metric, F.Cu at (142.5, 69.7)
- added C101: 10uF, Capacitor_SMD:C_0603_1608Metric, F.Cu at (142.5, 72.2)
- added C102: 4.7uF, Capacitor_SMD:C_0402_1005Metric, F.Cu at (144.6, 84.5)
- added C103: 47nF, Capacitor_SMD:C_0402_1005Metric, F.Cu at (144.6, 86.5)
- added C104: 10uF, Capacitor_SMD:C_0603_1608Metric, F.Cu at (142.5, 74.7)
- added C105: 100pF, Capacitor_SMD:C_0402_1005Metric, F.Cu at (144.6, 88.5)
- added C106: 100nF, Capacitor_SMD:C_0402_1005Metric, F.Cu at (144.6, 90.4)
- added C107: 10uF, Capacitor_SMD:C_0603_1608Metric, F.Cu at (142.5, 77.2)
- added C108: 100nF, Capacitor_SMD:C_0402_1005Metric, F.Cu at (166.7, 118.0)
- added C109: 1uF, Capacitor_SMD:C_0402_1005Metric, F.Cu at (166.7, 120.0)
- added C110: 100nF, Capacitor_SMD:C_0402_1005Metric, F.Cu at (166.7, 122.0)
- added C111: 100nF, Capacitor_SMD:C_0402_1005Metric, F.Cu at (166.7, 123.9)
- added C112: 100nF, Capacitor_SMD:C_0402_1005Metric, F.Cu at (166.7, 125.9)
- added C113: 10nF, Capacitor_SMD:C_0402_1005Metric, F.Cu at (144.6, 92.4)
- added C114: 6.8pF, Capacitor_SMD:C_0402_1005Metric, F.Cu at (180.4, 122.7)
- added C115: 6.8pF, Capacitor_SMD:C_0402_1005Metric, F.Cu at (180.4, 124.7)
- added C116: 10nF, Capacitor_SMD:C_0402_1005Metric, F.Cu at (180.4, 126.6)
- added C19: 1uF, Capacitor_SMD:C_0402_1005Metric, F.Cu at (174.8, 96.2)
- added C24: 1uF, Capacitor_SMD:C_0402_1005Metric, F.Cu at (174.8, 98.2)
- added C25: 1uF, Capacitor_SMD:C_0402_1005Metric, F.Cu at (174.8, 100.2)
- added C26: 1uF, Capacitor_SMD:C_0402_1005Metric, F.Cu at (174.8, 102.1)
- added C27: 1uF, Capacitor_SMD:C_0402_1005Metric, F.Cu at (174.8, 104.1)
- added C28: 1uF, Capacitor_SMD:C_0402_1005Metric, F.Cu at (174.8, 106.1)
- added C29: 1uF, Capacitor_SMD:C_0402_1005Metric, F.Cu at (174.8, 108.0)
- added C30: 1uF, Capacitor_SMD:C_0402_1005Metric, F.Cu at (177.7, 94.2)
- added C31: 1uF, Capacitor_SMD:C_0402_1005Metric, F.Cu at (177.7, 96.2)
- added C32: 1uF, Capacitor_SMD:C_0402_1005Metric, F.Cu at (177.7, 98.2)
- added C33: 1uF, Capacitor_SMD:C_0402_1005Metric, F.Cu at (177.7, 100.2)
- added C34: 1uF, Capacitor_SMD:C_0402_1005Metric, F.Cu at (177.7, 102.1)
- added C35: 1uF, Capacitor_SMD:C_0402_1005Metric, F.Cu at (177.7, 104.1)
- added C36: 1uF, Capacitor_SMD:C_0402_1005Metric, F.Cu at (177.7, 106.1)
- added C37: 1uF, Capacitor_SMD:C_0402_1005Metric, F.Cu at (177.7, 108.0)
- added C38: 1uF, Capacitor_SMD:C_0402_1005Metric, F.Cu at (180.5, 94.2)
- added C39: 1uF, Capacitor_SMD:C_0402_1005Metric, F.Cu at (180.5, 96.2)
- added C40: 1uF, Capacitor_SMD:C_0402_1005Metric, F.Cu at (180.5, 98.2)
- added C41: 1nF, Capacitor_SMD:C_0402_1005Metric, F.Cu at (180.5, 100.2)
- added C42: 1nF, Capacitor_SMD:C_0402_1005Metric, F.Cu at (180.5, 102.1)
- added C43: 1uF, Capacitor_SMD:C_0402_1005Metric, F.Cu at (180.5, 104.1)
- added C44: 1uF, Capacitor_SMD:C_0402_1005Metric, F.Cu at (180.5, 106.1)
- added C45: 1uF, Capacitor_SMD:C_0402_1005Metric, F.Cu at (180.5, 108.0)
- added C46: 1uF, Capacitor_SMD:C_0402_1005Metric, F.Cu at (183.4, 94.2)
- added C47: 1uF, Capacitor_SMD:C_0402_1005Metric, F.Cu at (183.4, 96.2)
- added C48: 1uF, Capacitor_SMD:C_0402_1005Metric, F.Cu at (183.4, 98.2)
- added C49: 1uF, Capacitor_SMD:C_0402_1005Metric, F.Cu at (183.4, 100.2)
- added C50: 1uF, Capacitor_SMD:C_0402_1005Metric, F.Cu at (183.4, 102.1)
- added C51: 2.2uF, Capacitor_SMD:C_0402_1005Metric, F.Cu at (183.4, 104.1)
- added C52: 2.2uF, Capacitor_SMD:C_0402_1005Metric, F.Cu at (183.4, 106.1)
- added C53: 1uF, Capacitor_SMD:C_0402_1005Metric, F.Cu at (183.4, 108.0)
- added C54: 2.2uF, Capacitor_SMD:C_0402_1005Metric, F.Cu at (186.3, 94.2)
- added C55: 1uF, Capacitor_SMD:C_0402_1005Metric, F.Cu at (186.3, 96.2)
- added C56: 100nF, Capacitor_SMD:C_0402_1005Metric, F.Cu at (186.3, 98.2)
- added C57: 1uF, Capacitor_SMD:C_0402_1005Metric, F.Cu at (186.3, 100.2)
- added C58: 1uF, Capacitor_SMD:C_0402_1005Metric, F.Cu at (186.3, 102.1)
- added C59: 100nF, Capacitor_SMD:C_0402_1005Metric, F.Cu at (186.3, 104.1)
- added C60: 100nF, Capacitor_SMD:C_0402_1005Metric, F.Cu at (135.8, 121.2)
- added C61: 100nF, Capacitor_SMD:C_0402_1005Metric, F.Cu at (135.8, 123.2)
- added C62: 100nF, Capacitor_SMD:C_0402_1005Metric, F.Cu at (135.8, 125.1)
- added C63: 100nF, Capacitor_SMD:C_0402_1005Metric, F.Cu at (135.8, 127.1)
- added C64: 100nF, Capacitor_SMD:C_0402_1005Metric, F.Cu at (135.8, 129.1)
- added C65: 100nF, Capacitor_SMD:C_0402_1005Metric, F.Cu at (135.8, 131.0)
- added C66: 100nF, Capacitor_SMD:C_0402_1005Metric, F.Cu at (135.8, 133.0)
- added C67: 100nF, Capacitor_SMD:C_0402_1005Metric, F.Cu at (135.8, 135.0)
- added C68: 100nF, Capacitor_SMD:C_0402_1005Metric, F.Cu at (138.7, 121.2)
- added C69: 100nF, Capacitor_SMD:C_0402_1005Metric, F.Cu at (138.7, 123.2)
- added C70: 100nF, Capacitor_SMD:C_0402_1005Metric, F.Cu at (138.7, 125.1)
- added C71: 100nF, Capacitor_SMD:C_0402_1005Metric, F.Cu at (138.7, 127.1)
- added C72: 100nF, Capacitor_SMD:C_0402_1005Metric, F.Cu at (138.7, 129.1)
- added C73: 100nF, Capacitor_SMD:C_0402_1005Metric, F.Cu at (138.7, 131.0)
- added C74: 100nF, Capacitor_SMD:C_0402_1005Metric, F.Cu at (138.7, 133.0)
- added C75: 100nF, Capacitor_SMD:C_0402_1005Metric, F.Cu at (138.7, 135.0)
- added C76: 100nF, Capacitor_SMD:C_0402_1005Metric, F.Cu at (141.5, 121.2)
- added C77: 100nF, Capacitor_SMD:C_0402_1005Metric, F.Cu at (141.5, 123.2)
- added C78: 100nF, Capacitor_SMD:C_0402_1005Metric, F.Cu at (141.5, 125.1)
- added C79: 100nF, Capacitor_SMD:C_0402_1005Metric, F.Cu at (141.5, 127.1)
- added C80: 100nF, Capacitor_SMD:C_0402_1005Metric, F.Cu at (141.5, 129.1)
- added C81: 100nF, Capacitor_SMD:C_0402_1005Metric, F.Cu at (141.5, 131.0)
- added C82: 100nF, Capacitor_SMD:C_0402_1005Metric, F.Cu at (141.5, 133.0)
- added C83: 100nF, Capacitor_SMD:C_0402_1005Metric, F.Cu at (141.5, 135.0)
- added C84: 100nF, Capacitor_SMD:C_0402_1005Metric, F.Cu at (144.4, 121.2)
- added C85: 1uF, Capacitor_SMD:C_0402_1005Metric, F.Cu at (144.4, 123.2)
- added C86: 1uF, Capacitor_SMD:C_0402_1005Metric, F.Cu at (144.4, 125.1)
- added C87: 10uF, Capacitor_SMD:C_0603_1608Metric, F.Cu at (125.3, 122.6)
- added C88: 10uF, Capacitor_SMD:C_0603_1608Metric, F.Cu at (125.3, 125.1)
- added C89: 100nF, Capacitor_SMD:C_0402_1005Metric, F.Cu at (144.4, 127.1)
- added C90: 4.7uF, Capacitor_SMD:C_0402_1005Metric, F.Cu at (166.7, 116.0)
- added C91: 10nF, Capacitor_SMD:C_0402_1005Metric, F.Cu at (167.5, 79.6)
- added C92: 6.8pF, Capacitor_SMD:C_0402_1005Metric, F.Cu at (167.5, 81.6)
- added C93: 6.8pF, Capacitor_SMD:C_0402_1005Metric, F.Cu at (167.5, 83.6)
- added C94: 10nF, Capacitor_SMD:C_0402_1005Metric, F.Cu at (167.5, 85.5)
- added C95: 10nF, Capacitor_SMD:C_0402_1005Metric, F.Cu at (167.5, 87.5)
- added C96: 1uF, Capacitor_SMD:C_0402_1005Metric, F.Cu at (141.7, 92.4)
- added C97: 220nF, Capacitor_SMD:C_0402_1005Metric, F.Cu at (141.7, 94.4)
- added C98: 10uF, Capacitor_SMD:C_0603_1608Metric, F.Cu at (138.5, 79.8)
- added C99: 10uF, Capacitor_SMD:C_0603_1608Metric, F.Cu at (138.5, 82.3)
- added D2: LED_R, LED_SMD:LED_0402_1005Metric, F.Cu at (183.5, 125.5)
- added D3: LED_B, LED_SMD:LED_0402_1005Metric, F.Cu at (183.5, 127.5)
- added D4: LED_B, LED_SMD:LED_0402_1005Metric, F.Cu at (148.7, 96.3)
- added D5: LED_R, LED_SMD:LED_0402_1005Metric, F.Cu at (148.7, 98.3)
- added D6: SMAJ5.0A, Diode_SMD:D_SMA, F.Cu at (127.4, 97.0)
- added J3: USB4215-03-A_REVA, lib:GCT_USB4215-03-A_REVA, F.Cu at (103.7, 120.0)
- added JP1: SolderJumper_3_Bridged12, Jumper:SolderJumper-3_P1.3mm_Bridged12_Pad1.0x1.5mm, F.Cu at (163.2, 80.4)
- added JP2: SolderJumper_3_Bridged12, Jumper:SolderJumper-3_P1.3mm_Bridged12_Pad1.0x1.5mm, F.Cu at (163.2, 84.2)
- added JP3: SolderJumper_3_Bridged12, Jumper:SolderJumper-3_P1.3mm_Bridged12_Pad1.0x1.5mm, F.Cu at (163.2, 88.1)
- added JP4: SolderJumper_3_Bridged12, Jumper:SolderJumper-3_P1.3mm_Bridged12_Pad1.0x1.5mm, F.Cu at (148.8, 85.3)
- added L5: 1uH, Inductor_SMD:L_0201_0603Metric, F.Cu at (180.1, 109.9)
- added L6: 1uH, Inductor_SMD:L_1008_2520Metric, F.Cu at (134.9, 100.4)
- added R1: 240, Resistor_SMD:R_0402_1005Metric, F.Cu at (135.8, 105.3)
- added R10: 56, Resistor_SMD:R_0402_1005Metric, F.Cu at (138.7, 107.3)
- added R11: 56, Resistor_SMD:R_0402_1005Metric, F.Cu at (138.7, 109.2)
- added R12: 56, Resistor_SMD:R_0402_1005Metric, F.Cu at (138.7, 111.2)
- added R13: 56, Resistor_SMD:R_0402_1005Metric, F.Cu at (138.7, 113.2)
- added R14: 56, Resistor_SMD:R_0402_1005Metric, F.Cu at (138.7, 115.2)
- added R15: 56, Resistor_SMD:R_0402_1005Metric, F.Cu at (138.7, 117.2)
- added R16: 56, Resistor_SMD:R_0402_1005Metric, F.Cu at (138.7, 119.2)
- added R17: 56, Resistor_SMD:R_0402_1005Metric, F.Cu at (141.6, 105.3)
- added R18: 56, Resistor_SMD:R_0402_1005Metric, F.Cu at (141.6, 107.3)
- added R19: 56, Resistor_SMD:R_0402_1005Metric, F.Cu at (141.6, 109.2)
- added R2: 100, Resistor_SMD:R_0402_1005Metric, F.Cu at (135.8, 107.3)
- added R20: 56, Resistor_SMD:R_0402_1005Metric, F.Cu at (141.6, 111.2)
- added R21: 56, Resistor_SMD:R_0402_1005Metric, F.Cu at (141.6, 113.2)
- added R22: 56, Resistor_SMD:R_0402_1005Metric, F.Cu at (141.6, 115.2)
- added R23: 56, Resistor_SMD:R_0402_1005Metric, F.Cu at (141.6, 117.2)
- added R24: 56, Resistor_SMD:R_0402_1005Metric, F.Cu at (141.6, 119.2)
- added R25: 56, Resistor_SMD:R_0402_1005Metric, F.Cu at (144.6, 105.3)
- added R26: 56, Resistor_SMD:R_0402_1005Metric, F.Cu at (144.6, 107.3)
- added R27: 56, Resistor_SMD:R_0402_1005Metric, F.Cu at (144.6, 109.2)
- added R28: 56, Resistor_SMD:R_0402_1005Metric, F.Cu at (144.6, 111.2)
- added R29: 240, Resistor_SMD:R_0402_1005Metric, F.Cu at (144.6, 113.2)
- added R3: 10k, Resistor_SMD:R_0402_1005Metric, F.Cu at (135.8, 109.2)
- added R30: 0, Resistor_SMD:R_0402_1005Metric, F.Cu at (169.5, 116.1)
- added R31: 10, Resistor_SMD:R_0402_1005Metric, F.Cu at (170.4, 86.3)
- added R32: 10k, Resistor_SMD:R_0402_1005Metric, F.Cu at (170.4, 88.3)
- added R33: 0, Resistor_SMD:R_0402_1005Metric, F.Cu at (170.4, 90.3)
- added R34: 1k, Resistor_SMD:R_0402_1005Metric, F.Cu at (173.3, 86.3)
- added R37: 10k, Resistor_SMD:R_0402_1005Metric, F.Cu at (173.3, 88.3)
- added R38: 10k, Resistor_SMD:R_0402_1005Metric, F.Cu at (173.3, 90.3)
- added R39: 10k, Resistor_SMD:R_0402_1005Metric, F.Cu at (176.2, 86.3)
- added R4: 10k, Resistor_SMD:R_0402_1005Metric, F.Cu at (135.8, 111.2)
- added R40: 0, Resistor_SMD:R_0402_1005Metric, F.Cu at (124.8, 87.8)
- added R41: 10k, Resistor_SMD:R_0402_1005Metric, F.Cu at (176.2, 88.3)
- added R42: 100, Resistor_SMD:R_0402_1005Metric, F.Cu at (176.2, 90.3)
- added R43: ~, Resistor_SMD:R_0402_1005Metric, F.Cu at (174.4, 116.1)
- added R44: ~, Resistor_SMD:R_0402_1005Metric, F.Cu at (174.4, 118.0)
- added R45: 10m, Resistor_SMD:R_0603_1608Metric, F.Cu at (142.5, 79.8)
- added R46: 1k, Resistor_SMD:R_0402_1005Metric, F.Cu at (124.8, 89.8)
- added R47: 1k, Resistor_SMD:R_0402_1005Metric, F.Cu at (124.8, 91.7)
- added R48: 2k2, Resistor_SMD:R_0402_1005Metric, F.Cu at (124.8, 93.7)
- added R49: 2k2, Resistor_SMD:R_0402_1005Metric, F.Cu at (127.7, 87.8)
- added R5: 56, Resistor_SMD:R_0402_1005Metric, F.Cu at (135.8, 113.2)
- added R50: 220, Resistor_SMD:R_0402_1005Metric, F.Cu at (127.7, 89.8)
- added R51: 10k, Resistor_SMD:R_0402_1005Metric, F.Cu at (127.7, 91.7)
- added R52: 5k23, Resistor_SMD:R_0402_1005Metric, F.Cu at (127.7, 93.7)
- added R53: 30k1, Resistor_SMD:R_0402_1005Metric, F.Cu at (130.6, 87.8)
- added R54: 240, Resistor_SMD:R_0402_1005Metric, F.Cu at (130.6, 89.8)
- added R55: 10k, Resistor_SMD:R_0402_1005Metric, F.Cu at (169.5, 118.0)
- added R56: 10k, Resistor_SMD:R_0402_1005Metric, F.Cu at (169.5, 120.0)
- added R57: 10k, Resistor_SMD:R_0402_1005Metric, F.Cu at (169.5, 122.0)
- added R58: 10k, Resistor_SMD:R_0402_1005Metric, F.Cu at (130.6, 91.7)
- added R59: 10k, Resistor_SMD:R_0402_1005Metric, F.Cu at (130.6, 93.7)
- added R6: 56, Resistor_SMD:R_0402_1005Metric, F.Cu at (135.8, 115.2)
- added R60: 4k7, Resistor_SMD:R_0402_1005Metric, F.Cu at (174.4, 120.0)
- added R61: 4k7, Resistor_SMD:R_0402_1005Metric, F.Cu at (174.4, 122.0)
- added R62: 3k, Resistor_SMD:R_0402_1005Metric, F.Cu at (174.4, 131.5)
- added R63: 10k, Resistor_SMD:R_0402_1005Metric, F.Cu at (174.4, 124.0)
- added R7: 56, Resistor_SMD:R_0402_1005Metric, F.Cu at (135.8, 117.2)
- added R8: 56, Resistor_SMD:R_0402_1005Metric, F.Cu at (135.8, 119.2)
- added R9: 56, Resistor_SMD:R_0402_1005Metric, F.Cu at (138.7, 105.3)
- added S1: DS04-254-2-03BK-SMT, lib:SW_DS04-254-2-03BK-SMT, F.Cu at (166.8, 73.5)
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Connections:
- net 5V_VIN renamed VIN
- C18 pad 1: unconnected-(C18-Pad1) -> GND
- U2 pad A1: unconnected-(U2A-VSS-PadA1) -> GND
- U2 pad A10: unconnected-(U2C-PC9-PadA10) -> SDMMC1_D1
- U2 pad A11: unconnected-(U2C-PC11-PadA11) -> SDMMC1_D3
- U2 pad A12: unconnected-(U2A-VDD_DSI-PadA12) -> VDD
- U2 pad A16: unconnected-(U2A-VDD1V2_DSI_PHY-PadA16) -> Net-(U2A-VDD1V2_DSI_PHY)
- U2 pad A17: unconnected-(U2B-DDR_DQ0-PadA17) -> /DDR/DDR_DQ0
- U2 pad A18: unconnected-(U2B-DDR_DQ1-PadA18) -> /DDR/DDR_DQ1
- U2 pad A19: unconnected-(U2A-VSS-PadA19) -> GND
- U2 pad A3: unconnected-(U2C-PD0-PadA3) -> NAND_D2
- U2 pad A4: unconnected-(U2C-PD1-PadA4) -> NAND_D3
- U2 pad B10: unconnected-(U2C-PD2-PadB10) -> SDMMC1_CMD
- U2 pad B12: unconnected-(U2A-VDDA1V8_DSI-PadB12) -> Net-(U2A-VDDA1V8_DSI)
- U2 pad B16: unconnected-(U2A-VDD1V2_DSI_REG-PadB16) -> Net-(U2A-VDD1V2_DSI_PHY)
- U2 pad B17: unconnected-(U2B-DDR_DQ3-PadB17) -> /DDR/DDR_DQ3
- U2 pad B18: unconnected-(U2B-DDR_DQ7-PadB18) -> /DDR/DDR_DQ7
- U2 pad B19: unconnected-(U2B-DDR_DQS0N-PadB19) -> /DDR/DDR_DQS0_N
- U2 pad B2: unconnected-(U2A-VSS-PadB2) -> GND
- U2 pad B5: unconnected-(U2C-PB7-PadB5) -> uSD_DETECT
- U2 pad B6: unconnected-(U2A-VSS-PadB6) -> GND
- U2 pad C10: unconnected-(U2C-PC12-PadC10) -> SDMMC1_CK
- U2 pad C11: unconnected-(U2C-PC8-PadC11) -> SDMMC1_D0
- U2 pad C12: unconnected-(U2A-VSS_DSI-PadC12) -> GND
- U2 pad C13: unconnected-(U2A-VSS_DSI-PadC13) -> GND
- U2 pad C14: unconnected-(U2A-VSS_DSI-PadC14) -> GND
- U2 pad C15: unconnected-(U2A-VSS_DSI-PadC15) -> GND
- U2 pad C16: unconnected-(U2A-VSS_DSI-PadC16) -> GND
- U2 pad C17: unconnected-(U2A-VSS-PadC17) -> GND
- U2 pad C18: unconnected-(U2B-DDR_DQM0-PadC18) -> /DDR/DDR_DQM0
- U2 pad C19: unconnected-(U2B-DDR_DQS0P-PadC19) -> /DDR/DDR_DQS0_P
- U2 pad C3: unconnected-(U2A-VSS-PadC3) -> GND
- U2 pad D1: unconnected-(U2A-VSS-PadD1) -> GND
- U2 pad D11: unconnected-(U2C-PC10-PadD11) -> SDMMC1_D2
- U2 pad D13: unconnected-(U2E-JTDI-PadD13) -> /RCC_BOOT_RST_DEBUG/T_JTDI/NC
- U2 pad D14: unconnected-(U2E-JTDO-PadD14) -> /RCC_BOOT_RST_DEBUG/T_JTDO/T_SWO
- U2 pad D15: unconnected-(U2E-JTMS-PadD15) -> /RCC_BOOT_RST_DEBUG/T_JTMS/T_SWDIO
- U2 pad D16: unconnected-(U2E-JTCK-PadD16) -> /RCC_BOOT_RST_DEBUG/T_JCLK/T_SWCLK
- U2 pad D17: unconnected-(U2B-DDR_DQ5-PadD17) -> /DDR/DDR_DQ5
- U2 pad D18: unconnected-(U2B-DDR_DQ2-PadD18) -> /DDR/DDR_DQ2
- U2 pad D19: unconnected-(U2B-DDR_DQ6-PadD19) -> /DDR/DDR_DQ6
- U2 pad D4: unconnected-(U2A-VSS-PadD4) -> GND
- U2 pad D5: unconnected-(U2A-VSS-PadD5) -> GND
- U2 pad D6: unconnected-(U2C-PD4-PadD6) -> NAND_NOE
- U2 pad D7: unconnected-(U2C-PD5-PadD7) -> NAND_NWE
- U2 pad D8: unconnected-(U2A-VSS-PadD8) -> GND
- U2 pad E10: unconnected-(U2A-VSS-PadE10) -> GND
- U2 pad E12: unconnected-(U2A-VSS-PadE12) -> GND
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Routing:
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Other:
- board outline added: 50 x 50 mm

Commit message: PCB_UPDATE
Parts:
- removed C108, C110, C111, C112: 100nF, Capacitor_SMD:C_0402_1005Metric
- removed C109: 1uF, Capacitor_SMD:C_0402_1005Metric
- removed R55, R56, R57: 10k, Resistor_SMD:R_0402_1005Metric
- added C117: 2.2uF, Capacitor_SMD:C_0402_1005Metric, F.Cu at (88.1, 83.7)
- added C118: 100nF, Capacitor_SMD:C_0402_1005Metric, F.Cu at (88.1, 85.7)
- added C119: 1uF, Capacitor_SMD:C_0402_1005Metric, F.Cu at (88.1, 87.6)
- added C120: 100nF, Capacitor_SMD:C_0402_1005Metric, F.Cu at (88.1, 89.6)
- added C121: 2.2uF, Capacitor_SMD:C_0402_1005Metric, F.Cu at (88.1, 91.6)
- added C122: 100nF, Capacitor_SMD:C_0402_1005Metric, F.Cu at (88.1, 93.5)
- added C123: 2.2uF, Capacitor_SMD:C_0402_1005Metric, F.Cu at (88.1, 95.5)
- added JP5: SolderJumper_2_Open, Jumper:SolderJumper-2_P1.3mm_Open_Pad1.0x1.5mm, F.Cu at (83.0, 96.4)
- added R64: 47k, Resistor_SMD:R_0402_1005Metric, F.Cu at (82.3, 83.7)
- added R65: 47k, Resistor_SMD:R_0402_1005Metric, F.Cu at (82.3, 85.7)
- added R66: 47k, Resistor_SMD:R_0402_1005Metric, F.Cu at (82.3, 87.7)
- added R67: 47k, Resistor_SMD:R_0402_1005Metric, F.Cu at (82.3, 89.7)
- added R68: 47k, Resistor_SMD:R_0402_1005Metric, F.Cu at (82.3, 91.7)
- added R69: 47k, Resistor_SMD:R_0402_1005Metric, F.Cu at (82.3, 93.6)
- added R70: 47k, Resistor_SMD:R_0402_1005Metric, F.Cu at (85.2, 83.7)
- added R71: 47k, Resistor_SMD:R_0402_1005Metric, F.Cu at (85.2, 85.7)
- added R72: 47k, Resistor_SMD:R_0402_1005Metric, F.Cu at (85.2, 87.7)
- added R73: 47k, Resistor_SMD:R_0402_1005Metric, F.Cu at (85.2, 89.7)
- added R74: 22, Resistor_SMD:R_0402_1005Metric, F.Cu at (85.2, 91.7)
- added U13: EMMC04G-W627-M06U, lib:BGA153N50P14X14_1300X1150X100N, F.Cu at (86.5, 68.7)
- U2: footprint lib:BGA354C80P19X19_1600X1600X129 -> Package_BGA:ST_LFBGA-354_16x16mm_Layout19x19_P0.8mm
- U8: value MT29F4G08ABBDAH4_D -> LBEE5PK2AE-771; footprint lib:BGA63C80P10X12_900X1100X100N -> lib:XCVR_LBEE5PK2AE-771
Connections:
- U2 pad A3: NAND_D2 -> unconnected-(U2C-PD0-PadA3)
- U2 pad A4: NAND_D3 -> unconnected-(U2C-PD1-PadA4)
- U2 pad A5: unconnected-(U2D-PE3-PadA5) -> SDMMC2_CK
- U2 pad A6: unconnected-(U2D-PG6-PadA6) -> SDMMC2_CMD
- U2 pad A7: unconnected-(U2C-PB3-PadA7) -> SDMMC2_D2
- U2 pad A8: unconnected-(U2C-PB15-PadA8) -> SDMMC2_D1
- U2 pad B7: unconnected-(U2D-PE5-PadB7) -> SDMMC2_D6
- U2 pad B8: unconnected-(U2C-PA8-PadB8) -> SDMMC2_D4
- U2 pad B9: unconnected-(U2C-PB4-PadB9) -> SDMMC2_D3
- U2 pad C6: unconnected-(U2C-PD3-PadC6) -> SDMMC2_D7
- U2 pad C8: unconnected-(U2C-PA9-PadC8) -> SDMMC2_D5
- U2 pad C9: unconnected-(U2C-PB14-PadC9) -> SDMMC2_D0
- U2 pad D6: NAND_NOE -> unconnected-(U2C-PD4-PadD6)
- U2 pad D7: NAND_NWE -> unconnected-(U2C-PD5-PadD7)
- U2 pad E3: NAND_NWAIT -> unconnected-(U2C-PD6-PadE3)
- U2 pad F3: NAND_D0 -> unconnected-(U2C-PD14-PadF3)
- U2 pad G1: NAND_D1 -> unconnected-(U2C-PD15-PadG1)
- U2 pad T10: NAND_D4 -> unconnected-(U2D-PE7-PadT10)
- U2 pad T11: NAND_D5 -> unconnected-(U2D-PE8-PadT11)
- U2 pad T14: NAND_NCE -> unconnected-(U2D-PG9-PadT14)
- U2 pad U11: NAND_ALE -> unconnected-(U2C-PD12-PadU11)
- U2 pad V10: NAND_D7 -> unconnected-(U2D-PE10-PadV10)
- U2 pad V8: NAND_CLE -> unconnected-(U2C-PD11-PadV8)
- U2 pad W7: NAND_D6 -> unconnected-(U2D-PE9-PadW7)

Commit message: wifi done
Parts:
- removed JP1, JP2, JP3, JP4: SolderJumper_3_Bridged12, Jumper:SolderJumper-3_P1.3mm_Bridged12_Pad1.0x1.5mm
- added C108: 10uF, Capacitor_SMD:C_0603_1608Metric, F.Cu at (157.9, 54.5)
- added C109: 10uF, Capacitor_SMD:C_0603_1608Metric, F.Cu at (157.9, 57.0)
- added C110: 4.7uF, Capacitor_SMD:C_0402_1005Metric, F.Cu at (160.8, 48.2)
- added C124: 100nF, Capacitor_SMD:C_0402_1005Metric, F.Cu at (160.8, 50.1)
- added C125: 100nF, Capacitor_SMD:C_0402_1005Metric, F.Cu at (160.8, 52.1)
- added L7: 1uH, Inductor_SMD:L_Murata_DFE201610P, F.Cu at (157.7, 59.9)
- added R75: 47k, Resistor_SMD:R_0402_1005Metric, F.Cu at (148.6, 54.3)
- added R76: 47k, Resistor_SMD:R_0402_1005Metric, F.Cu at (148.6, 56.3)
- added R77: 47k, Resistor_SMD:R_0402_1005Metric, F.Cu at (148.6, 58.2)
- added R78: 47k, Resistor_SMD:R_0402_1005Metric, F.Cu at (151.5, 54.3)
- added R79: 47k, Resistor_SMD:R_0402_1005Metric, F.Cu at (151.5, 56.3)
- added R80: 22, Resistor_SMD:R_0402_1005Metric, F.Cu at (151.5, 58.2)
- added R81: 0, Resistor_SMD:R_0402_1005Metric, F.Cu at (154.4, 54.3)
- added R82: 0, Resistor_SMD:R_0402_1005Metric, F.Cu at (154.4, 56.3)
- added R83: 0, Resistor_SMD:R_0402_1005Metric, F.Cu at (154.4, 58.2)
- added R84: 0, Resistor_SMD:R_0402_1005Metric, F.Cu at (165.7, 48.2)
- added R85: 0, Resistor_SMD:R_0402_1005Metric, F.Cu at (165.7, 50.2)
- added R86: 0, Resistor_SMD:R_0402_1005Metric, F.Cu at (165.7, 52.1)
- added R87: 0, Resistor_SMD:R_0402_1005Metric, F.Cu at (165.7, 54.1)
- added R88: 0, Resistor_SMD:R_0402_1005Metric, F.Cu at (165.7, 56.1)
- added R89: 0, Resistor_SMD:R_0402_1005Metric, F.Cu at (165.7, 58.1)
- added R90: 0, Resistor_SMD:R_0402_1005Metric, F.Cu at (165.7, 62.1)
- added R91: 0, Resistor_SMD:R_0402_1005Metric, F.Cu at (165.7, 64.1)
- added S5: EVQ-9P701P, lib:SW_EVQ-9P701P, F.Cu at (191.8, 118.0)
- added TP33: TestPoint, TestPoint:TestPoint_Pad_D1.0mm, F.Cu at (148.7, 48.7)
- added TP34: TestPoint, TestPoint:TestPoint_Pad_D1.0mm, F.Cu at (148.7, 51.8)
- added TP35: TestPoint, TestPoint:TestPoint_Pad_D1.0mm, F.Cu at (151.7, 48.7)
- added TP36: TestPoint, TestPoint:TestPoint_Pad_D1.0mm, F.Cu at (151.7, 51.8)
- added TP37: TestPoint, TestPoint:TestPoint_Pad_D1.0mm, F.Cu at (154.8, 48.7)
- added TP38: TestPoint, TestPoint:TestPoint_Pad_D1.0mm, F.Cu at (154.8, 51.8)
- added TP39: TestPoint, TestPoint:TestPoint_Pad_D1.0mm, F.Cu at (157.8, 48.7)
- added TP40: TestPoint, TestPoint:TestPoint_Pad_D1.0mm, F.Cu at (157.8, 51.8)
Connections:
- U2 pad T15: Net-(JP1-C) -> unconnected-(U2E-BYPASS_REG1V8-PadT15)
- U8 pad 1: unconnected-(U8-GND-Pad1) -> VDD
- U8 pad 10: unconnected-(U8-BT_UART_TXD-Pad10) -> UART8_RX_STM
- U8 pad 11: unconnected-(U8-~{BT_UART_CTS}-Pad11) -> UART8_CTS_STM
- U8 pad 12: unconnected-(U8-BT_UART_RXD-Pad12) -> UART8_TX_STM
- U8 pad 13: unconnected-(U8-~{BT_UART_RTS}-Pad13) -> UART8_RTS_STM
- U8 pad 14: unconnected-(U8-GND-Pad14) -> VDD
- U8 pad 16: unconnected-(U8-GND-Pad16) -> VDD
- U8 pad 17: unconnected-(U8-BT_HOST_WAKE-Pad17) -> BT_HOST_WAKE
- U8 pad 2: unconnected-(U8-SR_VLX-Pad2) -> Net-(U8-SR_VLX)
- U8 pad 21: unconnected-(U8-GND-Pad21) -> VDD
- U8 pad 22: unconnected-(U8-WL_ANT-Pad22) -> Net-(U8-WL_ANT)
- U8 pad 23: unconnected-(U8-GND-Pad23) -> VDD
- U8 pad 24: unconnected-(U8-GND-Pad24) -> VDD
- U8 pad 27: unconnected-(U8-GND-Pad27) -> VDD
- U8 pad 28: unconnected-(U8-SDIO_CMD-Pad28) -> SDMMC3_CMD
- U8 pad 29: unconnected-(U8-SDIO_DATA_1-Pad29) -> SDMMC3_D1
- U8 pad 3: unconnected-(U8-VBAT-Pad3) -> 3V3
- U8 pad 30: unconnected-(U8-SDIO_DATA_0-Pad30) -> SDMMC3_D0
- U8 pad 31: unconnected-(U8-SDIO_DATA_3-Pad31) -> SDMMC3_D3
- U8 pad 32: unconnected-(U8-SDIO_DATA_2-Pad32) -> SDMMC3_D2
- U8 pad 33: unconnected-(U8-SDIO_CLK-Pad33) -> Net-(U8-SDIO_CLK)
- U8 pad 34: unconnected-(U8-GND-Pad34) -> VDD
- U8 pad 4: unconnected-(U8-WL_REG_EN-Pad4) -> WL_REG_EN
- U8 pad 41: unconnected-(U8-GND-Pad41) -> VDD
- U8 pad 42: unconnected-(U8-VDDIO-Pad42) -> VDD
- U8 pad 43: unconnected-(U8-VIN_LDO-Pad43) -> Net-(U8-VIN_LDO)
- U8 pad 49: unconnected-(U8-USB2_AVDD33-Pad49) -> 3V3
- U8 pad 5: unconnected-(U8-LPO_IN-Pad5) -> MCO1/WIFI_LPO_IN
- U8 pad 51: unconnected-(U8-BT_DEV_WAKE-Pad51) -> BT_DEV_WAKE
- U8 pad 52: unconnected-(U8-WL_HOST_WAKE-Pad52) -> WL_HOST_WAKE
- U8 pad 54: unconnected-(U8-STRAP_1-Pad54) -> GND
- U8 pad 55: unconnected-(U8-STRAP_2-Pad55) -> VDD
- U8 pad 56: unconnected-(U8-STRAP_0-Pad56) -> Net-(U8-STRAP_0)
- U8 pad 57: unconnected-(U8-GND-Pad57) -> VDD
- U8 pad 6: unconnected-(U8-BT_PCM_IN-Pad6) -> I2S3_SDI
- U8 pad 68: unconnected-(U8-BT_REG_EN-Pad68) -> BT_REG_EN
- U8 pad 69: unconnected-(U8-GND-Pad69) -> VDD
- U8 pad 7: unconnected-(U8-BT_PCM_CLK-Pad7) -> I2S3_CK
- U8 pad 70: unconnected-(U8-GND-Pad70) -> VDD
- U8 pad 71: unconnected-(U8-GND-Pad71) -> VDD
- U8 pad 72: unconnected-(U8-GND-Pad72) -> VDD
- U8 pad 73: unconnected-(U8-GND-Pad73) -> VDD
- U8 pad 74: unconnected-(U8-GND-Pad74) -> VDD
- U8 pad 75: unconnected-(U8-GND-Pad75) -> VDD
- U8 pad 76: unconnected-(U8-GND-Pad76) -> VDD
- U8 pad 77: unconnected-(U8-GND-Pad77) -> VDD
- U8 pad 8: unconnected-(U8-BT_PCM_SYNC-Pad8) -> I2S3_WS
- U8 pad 9: unconnected-(U8-BT_PCM_OUT-Pad9) -> I2S3_SDO

Commit message: PCB_UPDATE
Parts:
- removed C1: CPH3225A, lib:CAPCP3225X100N
- removed C10, C100, C101, C104, C107, C108, C109, C11, C12, C13, C15, C17, C87, C88, C98, C99: 10uF, Capacitor_SMD:C_0603_1608Metric
- removed C102, C110, C14, C2, C3, C4, C5, C6, C7, C90: 4.7uF, Capacitor_SMD:C_0402_1005Metric
- removed C103: 47nF, Capacitor_SMD:C_0402_1005Metric
- removed C105: 100pF, Capacitor_SMD:C_0402_1005Metric
- removed C106, C118, C120, C122, C124, C125, C56, C59, C60, C61, C62, C63, C64, C65, C66, C67, C68, C69, C70, C71, C72, C73, C74, C75, C76, C77, C78, C79, C80, C81, C82, C83, C84, C89: 100nF, Capacitor_SMD:C_0402_1005Metric
- removed C113, C116, C91, C94, C95: 10nF, Capacitor_SMD:C_0402_1005Metric
- removed C114, C115, C92, C93: 6.8pF, Capacitor_SMD:C_0402_1005Metric
- removed C117, C121, C123, C51, C52, C54: 2.2uF, Capacitor_SMD:C_0402_1005Metric
- removed C119, C16, C18, C19, C24, C25, C26, C27, C28, C29, C30, C31, C32, C33, C34, C35, C36, C37, C38, C39, C40, C43, C44, C45, C46, C47, C48, C49, C50, C53, C55, C57, C58, C8, C85, C86, C9, C96: 1uF, Capacitor_SMD:C_0402_1005Metric
- removed C20, C21, C22, C23: 22uF, Capacitor_SMD:C_0603_1608Metric
- removed C41, C42: 1nF, Capacitor_SMD:C_0402_1005Metric
- removed C97: 220nF, Capacitor_SMD:C_0402_1005Metric
- removed D2, D5: LED_R, LED_SMD:LED_0402_1005Metric
- removed D3, D4: LED_B, LED_SMD:LED_0402_1005Metric
- removed D6: SMAJ5.0A, Diode_SMD:D_SMA
- removed J3: USB4215-03-A_REVA, lib:GCT_USB4215-03-A_REVA
- removed JP5: SolderJumper_2_Open, Jumper:SolderJumper-2_P1.3mm_Open_Pad1.0x1.5mm
- removed L1, L2, L3, L4, L6: 1uH, Inductor_SMD:L_1008_2520Metric
- removed L5: 1uH, Inductor_SMD:L_0201_0603Metric
- removed L7: 1uH, Inductor_SMD:L_Murata_DFE201610P
- removed R1, R29, R54: 240, Resistor_SMD:R_0402_1005Metric
- removed R10, R11, R12, R13, R14, R15, R16, R17, R18, R19, R20, R21, R22, R23, R24, R25, R26, R27, R28, R5, R6, R7, R8, R9: 56, Resistor_SMD:R_0402_1005Metric
- removed R2, R42: 100, Resistor_SMD:R_0402_1005Metric
- removed R3, R32, R37, R38, R39, R4, R41, R51, R58, R59, R63: 10k, Resistor_SMD:R_0402_1005Metric
- removed R30, R33, R40, R81, R82, R83, R84, R85, R86, R87, R88, R89, R90, R91: 0, Resistor_SMD:R_0402_1005Metric
- removed R31: 10, Resistor_SMD:R_0402_1005Metric
- removed R34, R46, R47: 1k, Resistor_SMD:R_0402_1005Metric
- removed R43, R44: ~, Resistor_SMD:R_0402_1005Metric
- removed R45: 10m, Resistor_SMD:R_0603_1608Metric
- removed R48, R49: 2k2, Resistor_SMD:R_0402_1005Metric
- removed R50: 220, Resistor_SMD:R_0402_1005Metric
- removed R52: 5k23, Resistor_SMD:R_0402_1005Metric
- removed R53: 30k1, Resistor_SMD:R_0402_1005Metric
- removed R60, R61: 4k7, Resistor_SMD:R_0402_1005Metric
- removed R62: 3k, Resistor_SMD:R_0402_1005Metric
- removed R64, R65, R66, R67, R68, R69, R70, R71, R72, R73, R75, R76, R77, R78, R79: 47k, Resistor_SMD:R_0402_1005Metric
- removed R74, R80: 22, Resistor_SMD:R_0402_1005Metric
- removed S1: DS04-254-2-03BK-SMT, lib:SW_DS04-254-2-03BK-SMT
- removed S2, S3, S4: PTS525SM15SMTR2LFS, lib:SW_PTS525SM15SMTR2LFS
- removed S5: EVQ-9P701P, lib:SW_EVQ-9P701P
- removed TP1, TP10, TP11, TP12, TP13, TP14, TP15, TP16, TP17, TP18, TP19, TP2, TP20, TP21, TP22, TP23, TP24, TP25, TP26, TP27, TP28, TP29, TP3, TP30, TP31, TP32, TP33, TP34, TP35, TP36, TP37, TP38, TP39, TP4, TP40, TP5, TP6, TP7, TP8, TP9: TestPoint, TestPoint:TestPoint_Pad_D1.0mm
- removed U1: STPMIC1APQR, lib:QFN40P600X500X80-45N
- removed U10: BQ25606RGER, lib:QFN50P400X400X100-25N
- removed U11, U4, U5, U6, U7: HSP051-4M10, lib:IC_HSP051-4M10
- removed U13: EMMC04G-W627-M06U, lib:BGA153N50P14X14_1300X1150X100N
- removed U2: STM32MP157FABx, Package_BGA:ST_LFBGA-354_16x16mm_Layout19x19_P0.8mm
- removed U3: MT41K256M16TW-107_P, lib:BGA96C80P9X16_1400X800X120
- removed U8: LBEE5PK2AE-771, lib:XCVR_LBEE5PK2AE-771
- removed U9: STC3115IQT, lib:SON50P300X200X60-10N
- removed Y1: ECS-2520MVQ-240, Oscillator:Oscillator_SMD_ECS_2520MV-xxx-xx-4Pin_2.5x2.0mm
- removed Y2: NX2012SA-32.768K, lib:XTAL_NX2012SA-32.768K-STD-MUB-1
- added BT201: Battery_Cell, Connector_PinHeader_1.00mm:PinHeader_1x02_P1.00mm_Vertical, F.Cu at (135.6, 31.9)
- added C201: 10uF, Capacitor_SMD:C_0603_1608Metric, F.Cu at (128.5, 66.0)
- added C202: 10uF, Capacitor_SMD:C_0603_1608Metric, F.Cu at (128.5, 68.5)
- added C203: 10uF, Capacitor_SMD:C_0603_1608Metric, F.Cu at (128.5, 71.0)
- added C204: 220nF, Capacitor_SMD:C_0402_1005Metric, F.Cu at (139.9, 65.7)
- added C205: 1uF, Capacitor_SMD:C_0402_1005Metric, F.Cu at (139.9, 67.7)
- added C206: 47nF, Capacitor_SMD:C_0402_1005Metric, F.Cu at (139.9, 69.6)
- added C207: 4.7uF, Capacitor_SMD:C_0402_1005Metric, F.Cu at (139.9, 71.6)
- added C208: 10uF, Capacitor_SMD:C_0603_1608Metric, F.Cu at (128.5, 73.5)
- added C209: 10uF, Capacitor_SMD:C_0603_1608Metric, F.Cu at (128.5, 76.0)
- added C210: 10nF, Capacitor_SMD:C_0402_1005Metric, F.Cu at (139.9, 73.6)
- added C211: 10uF, Capacitor_SMD:C_0603_1608Metric, F.Cu at (128.5, 78.5)
- added C212: 10uF, Capacitor_SMD:C_0603_1608Metric, F.Cu at (132.5, 66.0)
- added C213: 10uF, Capacitor_SMD:C_0603_1608Metric, F.Cu at (132.5, 68.5)
- added C214: 10uF, Capacitor_SMD:C_0603_1608Metric, F.Cu at (132.5, 71.0)
- added C215: 10uF, Capacitor_SMD:C_0603_1608Metric, F.Cu at (132.5, 73.5)
- added C216: 1uF, Capacitor_SMD:C_0402_1005Metric, F.Cu at (139.9, 75.5)
- added C217: 1uF, Capacitor_SMD:C_0402_1005Metric, F.Cu at (142.8, 65.7)
- added C218: 4.7uF, Capacitor_SMD:C_0402_1005Metric, F.Cu at (142.8, 67.7)
- added C219: 1uF, Capacitor_SMD:C_0402_1005Metric, F.Cu at (142.8, 69.6)
- added C220: 4.7uF, Capacitor_SMD:C_0402_1005Metric, F.Cu at (142.8, 71.6)
- added C221: 4.7uF, Capacitor_SMD:C_0402_1005Metric, F.Cu at (142.8, 73.6)
- added C222: 10uF, Capacitor_SMD:C_0603_1608Metric, F.Cu at (132.5, 76.0)
- added C223: 4.7uF, Capacitor_SMD:C_0402_1005Metric, F.Cu at (142.8, 75.5)
- added C224: 4.7uF, Capacitor_SMD:C_0402_1005Metric, F.Cu at (145.7, 65.7)
- added C225: 4.7uF, Capacitor_SMD:C_0402_1005Metric, F.Cu at (145.7, 67.7)
- added C226: 4.7uF, Capacitor_SMD:C_0402_1005Metric, F.Cu at (145.7, 69.6)
- added C227: 22uF, Capacitor_SMD:C_0603_1608Metric, F.Cu at (132.5, 78.5)
- added C228: 22uF, Capacitor_SMD:C_0603_1608Metric, F.Cu at (136.5, 66.0)
- added C229: 22uF, Capacitor_SMD:C_0603_1608Metric, F.Cu at (136.5, 68.5)
- added C230: 22uF, Capacitor_SMD:C_0603_1608Metric, F.Cu at (136.5, 71.0)
- added C301: 1uF, Capacitor_SMD:C_0402_1005Metric, F.Cu at (142.0, 43.9)
- added C302: 1uF, Capacitor_SMD:C_0402_1005Metric, F.Cu at (142.0, 45.8)
- added C303: 1uF, Capacitor_SMD:C_0402_1005Metric, F.Cu at (142.0, 47.8)
- added C304: 1uF, Capacitor_SMD:C_0402_1005Metric, F.Cu at (142.0, 49.8)
- added C305: 1uF, Capacitor_SMD:C_0402_1005Metric, F.Cu at (142.0, 51.8)
- added C306: 1uF, Capacitor_SMD:C_0402_1005Metric, F.Cu at (142.0, 53.7)
- added C307: 1uF, Capacitor_SMD:C_0402_1005Metric, F.Cu at (142.0, 55.7)
- added C308: 1uF, Capacitor_SMD:C_0402_1005Metric, F.Cu at (142.0, 57.7)
- added C309: 1uF, Capacitor_SMD:C_0402_1005Metric, F.Cu at (144.9, 43.9)
- added C310: 1uF, Capacitor_SMD:C_0402_1005Metric, F.Cu at (144.9, 45.8)
- added C311: 1uF, Capacitor_SMD:C_0402_1005Metric, F.Cu at (144.9, 47.8)
- added C312: 1uF, Capacitor_SMD:C_0402_1005Metric, F.Cu at (144.9, 49.8)
- added C313: 1uF, Capacitor_SMD:C_0402_1005Metric, F.Cu at (144.9, 51.8)
- added C314: 1uF, Capacitor_SMD:C_0402_1005Metric, F.Cu at (144.9, 53.7)
- added C315: 1uF, Capacitor_SMD:C_0402_1005Metric, F.Cu at (144.9, 55.7)
- added C316: 1uF, Capacitor_SMD:C_0402_1005Metric, F.Cu at (144.9, 57.7)
- added C317: 1uF, Capacitor_SMD:C_0402_1005Metric, F.Cu at (147.8, 43.9)
- added C318: 1uF, Capacitor_SMD:C_0402_1005Metric, F.Cu at (147.8, 45.8)
- added C319: 1uF, Capacitor_SMD:C_0402_1005Metric, F.Cu at (147.8, 47.8)
- added C320: 1uF, Capacitor_SMD:C_0402_1005Metric, F.Cu at (147.8, 49.8)
- added C321: 1uF, Capacitor_SMD:C_0402_1005Metric, F.Cu at (147.8, 51.8)
- added C322: 1uF, Capacitor_SMD:C_0402_1005Metric, F.Cu at (147.8, 53.7)
- added C323: 1uF, Capacitor_SMD:C_0402_1005Metric, F.Cu at (147.8, 55.7)
- added C324: 1nF, Capacitor_SMD:C_0402_1005Metric, F.Cu at (147.8, 57.7)
- added C325: 1nF, Capacitor_SMD:C_0402_1005Metric, F.Cu at (150.6, 43.9)
- added C326: 1uF, Capacitor_SMD:C_0402_1005Metric, F.Cu at (150.6, 45.8)
- added C327: 100nF, Capacitor_SMD:C_0402_1005Metric, F.Cu at (150.6, 47.8)
- added C328: 1uF, Capacitor_SMD:C_0402_1005Metric, F.Cu at (150.6, 49.8)
- added C329: 1uF, Capacitor_SMD:C_0402_1005Metric, F.Cu at (150.6, 51.8)
- added C330: 1uF, Capacitor_SMD:C_0402_1005Metric, F.Cu at (150.6, 53.7)
- added C331: 1uF, Capacitor_SMD:C_0402_1005Metric, F.Cu at (150.6, 55.7)
- added C332: CPH3225A, lib:CAPCP3225X100N, F.Cu at (143.5, 60.7)
- added C333: 1uF, Capacitor_SMD:C_0402_1005Metric, F.Cu at (150.6, 57.7)
- added C334: 2.2uF, Capacitor_SMD:C_0402_1005Metric, F.Cu at (153.5, 43.9)
- added C335: 1uF, Capacitor_SMD:C_0402_1005Metric, F.Cu at (153.5, 45.8)
- added C336: 2.2uF, Capacitor_SMD:C_0402_1005Metric, F.Cu at (153.5, 47.8)
- added C337: 1uF, Capacitor_SMD:C_0402_1005Metric, F.Cu at (153.5, 49.8)
- added C338: 2.2uF, Capacitor_SMD:C_0402_1005Metric, F.Cu at (153.5, 51.8)
- added C339: 100nF, Capacitor_SMD:C_0402_1005Metric, F.Cu at (153.5, 53.7)
- added C401: 100nF, Capacitor_SMD:C_0402_1005Metric, F.Cu at (90.7, 39.2)
- added C402: 100nF, Capacitor_SMD:C_0402_1005Metric, F.Cu at (90.7, 41.1)
- added C403: 100nF, Capacitor_SMD:C_0402_1005Metric, F.Cu at (90.7, 43.1)
- added C404: 1uF, Capacitor_SMD:C_0402_1005Metric, F.Cu at (76.7, 70.5)
- added C405: 100nF, Capacitor_SMD:C_0402_1005Metric, F.Cu at (76.7, 72.4)
- added C406: 100nF, Capacitor_SMD:C_0402_1005Metric, F.Cu at (76.7, 74.4)
- added C407: 100nF, Capacitor_SMD:C_0402_1005Metric, F.Cu at (90.7, 51.0)
- added C408: 100nF, Capacitor_SMD:C_0402_1005Metric, F.Cu at (90.7, 53.0)
- added C409: 100nF, Capacitor_SMD:C_0402_1005Metric, F.Cu at (93.6, 39.2)
- added C410: 100nF, Capacitor_SMD:C_0402_1005Metric, F.Cu at (93.6, 41.1)
- added C411: 100nF, Capacitor_SMD:C_0402_1005Metric, F.Cu at (93.6, 43.1)
- added C412: 100nF, Capacitor_SMD:C_0402_1005Metric, F.Cu at (93.6, 45.1)
- added C413: 100nF, Capacitor_SMD:C_0402_1005Metric, F.Cu at (93.6, 47.0)
- added C414: 100nF, Capacitor_SMD:C_0402_1005Metric, F.Cu at (93.6, 49.0)
- added C415: 100nF, Capacitor_SMD:C_0402_1005Metric, F.Cu at (93.6, 51.0)
- added C416: 100nF, Capacitor_SMD:C_0402_1005Metric, F.Cu at (93.6, 53.0)
- added C417: 100nF, Capacitor_SMD:C_0402_1005Metric, F.Cu at (96.5, 39.2)
- added C418: 100nF, Capacitor_SMD:C_0402_1005Metric, F.Cu at (96.5, 41.1)
- added C419: 1uF, Capacitor_SMD:C_0402_1005Metric, F.Cu at (82.4, 68.5)
- added C420: 100nF, Capacitor_SMD:C_0402_1005Metric, F.Cu at (82.4, 70.5)
- added C421: 100nF, Capacitor_SMD:C_0402_1005Metric, F.Cu at (82.4, 72.4)
- added C422: 10uF, Capacitor_SMD:C_0603_1608Metric, F.Cu at (66.2, 66.0)
- added C423: 100nF, Capacitor_SMD:C_0402_1005Metric, F.Cu at (82.4, 74.4)
- added C424: 100nF, Capacitor_SMD:C_0402_1005Metric, F.Cu at (82.4, 76.4)
- added C425: 10uF, Capacitor_SMD:C_0603_1608Metric, F.Cu at (66.2, 68.5)
- added C426: 100nF, Capacitor_SMD:C_0402_1005Metric, F.Cu at (82.4, 78.3)
- added C427: 100nF, Capacitor_SMD:C_0402_1005Metric, F.Cu at (85.3, 64.5)
- added C428: 100nF, Capacitor_SMD:C_0402_1005Metric, F.Cu at (85.3, 66.5)
- added C429: 100nF, Capacitor_SMD:C_0402_1005Metric, F.Cu at (85.3, 68.5)
- added C430: 100nF, Capacitor_SMD:C_0402_1005Metric, F.Cu at (85.3, 70.5)
- added C501: 2.2uF, Capacitor_SMD:C_0402_1005Metric, F.Cu at (170.9, 81.7)
- added C502: 100nF, Capacitor_SMD:C_0402_1005Metric, F.Cu at (170.9, 83.7)
- added C503: 100nF, Capacitor_SMD:C_0402_1005Metric, F.Cu at (170.9, 85.7)
- added C504: 100nF, Capacitor_SMD:C_0402_1005Metric, F.Cu at (170.9, 87.6)
- added C505: 2.2uF, Capacitor_SMD:C_0402_1005Metric, F.Cu at (170.9, 89.6)
- added C506: 2.2uF, Capacitor_SMD:C_0402_1005Metric, F.Cu at (170.9, 91.6)
- added C507: 1uF, Capacitor_SMD:C_0402_1005Metric, F.Cu at (170.9, 93.5)
- added C508: 4.7uF, Capacitor_SMD:C_0402_1005Metric, F.Cu at (170.9, 95.5)
- added C601: 6.8pF, Capacitor_SMD:C_0402_1005Metric, F.Cu at (188.5, 120.3)
- added C602: 6.8pF, Capacitor_SMD:C_0402_1005Metric, F.Cu at (188.5, 122.3)
- added C701: 10nF, Capacitor_SMD:C_0402_1005Metric, F.Cu at (141.5, 112.1)
- added C702: 10nF, Capacitor_SMD:C_0402_1005Metric, F.Cu at (141.5, 114.1)
- added C703: 6.8pF, Capacitor_SMD:C_0402_1005Metric, F.Cu at (141.5, 116.0)
- added C704: 10nF, Capacitor_SMD:C_0402_1005Metric, F.Cu at (141.5, 118.0)
- added C705: 6.8pF, Capacitor_SMD:C_0402_1005Metric, F.Cu at (141.5, 120.0)
- added C801: 100nF, Capacitor_SMD:C_0402_1005Metric, F.Cu at (188.5, 53.1)
- added C802: 100nF, Capacitor_SMD:C_0402_1005Metric, F.Cu at (188.5, 55.1)
- added C803: 100pF, Capacitor_SMD:C_0402_1005Metric, F.Cu at (188.5, 57.1)
- added C804: 100nF, Capacitor_SMD:C_0402_1005Metric, F.Cu at (188.5, 59.0)
- added C805: 10uF, Capacitor_SMD:C_0603_1608Metric, F.Cu at (191.9, 53.4)
- added C901: 4.7uF, Capacitor_SMD:C_0402_1005Metric, F.Cu at (174.1, 55.9)
- added C902: 10uF, Capacitor_SMD:C_0603_1608Metric, F.Cu at (171.1, 44.1)
- added C903: 10uF, Capacitor_SMD:C_0603_1608Metric, F.Cu at (171.1, 46.6)
- added C904: 100nF, Capacitor_SMD:C_0402_1005Metric, F.Cu at (174.1, 57.9)
- added C905: 100nF, Capacitor_SMD:C_0402_1005Metric, F.Cu at (174.1, 59.9)
- added D201: LED_R, LED_SMD:LED_0402_1005Metric, F.Cu at (123.2, 89.1)
- added D202: LED_B, LED_SMD:LED_0402_1005Metric, F.Cu at (123.2, 91.1)
- added D203: PTVS3V3S1UR, lib:TVS_PTVS3V3S1UR, F.Cu at (137.4, 36.1)
- added D601: LED_B, LED_SMD:LED_0402_1005Metric, F.Cu at (188.7, 116.4)
- added D602: LED_R, LED_SMD:LED_0402_1005Metric, F.Cu at (188.7, 118.3)
- added D701: PTVS3V3S1UR, lib:TVS_PTVS3V3S1UR, F.Cu at (124.4, 40.5)
- added D801: ESDA7P120-1U1M, lib:DIODE_ESDA7P120-1U1M_STM, F.Cu at (191.5, 56.0)
- added J501: MEM2090-00-145-00-A_REVA, lib:GCT_MEM2090-00-145-00-A_REVA, F.Cu at (160.3, 80.7)
- added J701: FTSH-107-01-L-DV-K-A, lib:SAMTEC_FTSH-107-01-L-DV-K-A, F.Cu at (126.7, 34.6)
- added J801: USB4215-03-A_REVA, lib:GCT_USB4215-03-A_REVA, F.Cu at (183.6, 49.3)
- added J901: 73412-0110, lib:MOLEX_73412-0110, F.Cu at (169.9, 57.7)
- added L201: 1uH, Inductor_SMD:L_1008_2520Metric, F.Cu at (124.0, 66.6)
- added L202: 1uH, Inductor_SMD:L_1008_2520Metric, F.Cu at (124.0, 70.3)
- added L203: 1uH, Inductor_SMD:L_1008_2520Metric, F.Cu at (124.0, 74.1)
- added L204: 1uH, Inductor_SMD:L_1008_2520Metric, F.Cu at (124.0, 77.8)
- added L205: 1uH, Inductor_SMD:L_1008_2520Metric, F.Cu at (124.0, 81.6)
- added L301: 1uH, Inductor_SMD:L_0201_0603Metric, F.Cu at (147.3, 59.5)
- added L901: 1uH, Inductor_SMD:L_Murata_DFE201610P, F.Cu at (158.8, 60.0)
- added R201: 10k, Resistor_SMD:R_0402_1005Metric, F.Cu at (127.9, 80.8)
- added R202: 10k, Resistor_SMD:R_0402_1005Metric, F.Cu at (127.9, 82.7)
- added R203: 0, Resistor_SMD:R_0402_1005Metric, F.Cu at (127.9, 84.7)
- added R204: 2k2, Resistor_SMD:R_0402_1005Metric, F.Cu at (127.9, 86.7)
- added R205: 2k2, Resistor_SMD:R_0402_1005Metric, F.Cu at (127.9, 88.7)
- added R206: 220, Resistor_SMD:R_0402_1005Metric, F.Cu at (130.8, 80.8)
- added R207: 0, Resistor_SMD:R_0402_1005Metric, F.Cu at (130.8, 82.7)
- added R208: 10k, Resistor_SMD:R_0402_1005Metric, F.Cu at (130.8, 84.7)
- added R209: 1k, Resistor_SMD:R_0402_1005Metric, F.Cu at (130.8, 86.7)
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Routing:
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
Commit message: PCB_UPDATE
Parts:
- C403, C421, C422, C423, C427, C428, C429, R403, R404: moved to B.Cu
- moved R401 56.4 mm to (84.8, 79.3)
- moved R402 51.1 mm to (103.5, 74.7), turned to -90 degrees
- moved R405 49.6 mm to (115.8, 74.0)
- moved R404 46.0 mm to (102.5, 73.7), turned to 90 degrees
- moved R403 44.4 mm to (104.8, 69.3), turned to 180 degrees
- moved C425 43.9 mm to (109.5, 75.5), turned to 180 degrees
- moved C401 40.9 mm to (82.7, 79.3)
- moved C405 39.1 mm to (115.5, 67.8)
- moved C406 39.1 mm to (115.5, 69.8)
- moved C404 38.8 mm to (115.5, 71.3), turned to 180 degrees
- moved C402 35.0 mm to (102.1, 74.2)
- moved C420 33.3 mm to (115.4, 66.3)
- moved C422 32.1 mm to (98.0, 61.7), turned to 180 degrees
- moved C423 29.8 mm to (110.3, 64.0)
- moved U301 28.9 mm to (80.0, 69.0), turned to 0 degrees
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Connections:
- U401 pad A3: /DDR/DDR_DQ15 -> /DDR/DDR_DQ8
- U401 pad A7: /DDR/DDR_DQ12 -> /DDR/DDR_DQ15
- U401 pad B8: /DDR/DDR_DQ14 -> /DDR/DDR_DQ12
- U401 pad C2: /DDR/DDR_DQ11 -> /DDR/DDR_DQ10
- U401 pad C8: /DDR/DDR_DQ10 -> /DDR/DDR_DQ14
- U401 pad D7: /DDR/DDR_DQ8 -> /DDR/DDR_DQ11
Routing:
- net /DDR/DDR_DQS0_N: track 0.00 -> 33.1 mm
- net /DDR/DDR_DQS0_P: track 0.00 -> 33.0 mm
- net /DDR/DDR_DQ15: track 0.00 -> 29.8 mm
- net /DDR/DDR_DQ14: track 0.00 -> 28.5 mm
- net /DDR/DDR_DQ12: track 0.00 -> 27.4 mm
- net /DDR/DDR_DQM1: track 0.00 -> 26.3 mm
- net /DDR/DDR_DQ11: track 0.00 -> 26.1 mm
- net /DDR/DDR_DQS1_P: track 0.00 -> 22.2 mm
- net /DDR/DDR_DQS1_N: track 0.00 -> 21.5 mm
- net /DDR/DDR_A0: track 0.00 -> 1.47 mm
