File: PCB/MPU_MOD.kicad_pcb (KiCad board)
At the start: 2 copper layers, 50 x 50 mm, 294 parts, among them J501 MEM2090-00-145-00-A_REVA, J701 FTSH-107-01-L-DV-K-A, J801 USB4215-03-A_REVA, J901 73412-0110, U201 STC3115IQT, U202 BQ25606RGER, U203 STPMIC1APQR, U301 STM32MP157FABx, U401 MT41K256M16TW-107_P, U501 EMMC04G-W627-M06U, U502 HSP051-4M10, U503 HSP051-4M10, U701 HSP051-4M10, U702 HSP051-4M10, U801 FUSB302BMPX, U802 HSP051-4M10, U901 LBEE5PK2AE-771, Y601 NX2012SA-32.768K, Y701 ECS-2520MVQ-240

Commit message: PCB_UPDATE
Parts:
- moved C420 15.7 mm to (102.0, 74.5), turned to 180 degrees
- moved C403 3.11 mm to (101.8, 64.3)
- moved C428 3.11 mm to (103.6, 64.3)
- moved C430 3.11 mm to (106.1, 74.5)
- moved U401 3.11 mm to (101.2, 68.9)
- moved C402 3.11 mm to (99.0, 74.5)
- moved C421 3.11 mm to (105.4, 64.3)
- moved C422 3.11 mm to (94.9, 62.0)
- moved C423 3.11 mm to (107.2, 64.3)
- moved C424 3.11 mm to (97.2, 74.5)
- moved C425 3.11 mm to (106.4, 75.8)
- moved C426 3.11 mm to (95.4, 74.5)
- moved C427 3.11 mm to (106.0, 72.2)
- moved C429 3.11 mm to (95.5, 63.3)
- moved R402 3.11 mm to (100.4, 75.0)
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Connections:
- U401 pad A2: /DDR/DDR_DQ13 -> /DDR/DDR_DQ0
- U401 pad A3: /DDR/DDR_DQ8 -> /DDR/DDR_DQ7
- U401 pad A7: /DDR/DDR_DQ15 -> /DDR/DDR_DQ2
- U401 pad B8: /DDR/DDR_DQ12 -> /DDR/DDR_DQ4
- U401 pad C2: /DDR/DDR_DQ10 -> /DDR/DDR_DQ3
- U401 pad C3: /DDR/DDR_DQ9 -> /DDR/DDR_DQ1
- U401 pad C8: /DDR/DDR_DQ14 -> /DDR/DDR_DQ5
- U401 pad D7: /DDR/DDR_DQ11 -> /DDR/DDR_DQ6
- U401 pad E3: /DDR/DDR_DQ0 -> /DDR/DDR_DQ9
- U401 pad F2: /DDR/DDR_DQ2 -> /DDR/DDR_DQ8
- U401 pad F7: /DDR/DDR_DQ1 -> /DDR/DDR_DQ12
- U401 pad F8: /DDR/DDR_DQ3 -> /DDR/DDR_DQ15
- U401 pad G2: /DDR/DDR_DQ6 -> /DDR/DDR_DQ10
- U401 pad H3: /DDR/DDR_DQ4 -> /DDR/DDR_DQ13
- U401 pad H7: /DDR/DDR_DQ7 -> /DDR/DDR_DQ14
- U401 pad H8: /DDR/DDR_DQ5 -> /DDR/DDR_DQ11
Routing:
- net /DDR/DDR_DQM1: track 26.3 -> 0.00 mm
- net /DDR/DDR_DQ0: track 0.00 -> 24.8 mm, vias 0 -> 2
- net /DDR/DDR_DQ7: track 0.00 -> 23.6 mm, vias 0 -> 2
- net /DDR/DDR_DQ3: track 0.00 -> 23.2 mm, vias 0 -> 2
- net /DDR/DDR_DQ1: track 0.00 -> 21.8 mm, vias 0 -> 2
- net /DDR/DDR_DQ9: track 0.00 -> 21.6 mm
- net /DDR/DDR_DQ8: track 0.00 -> 21.4 mm
- net /DDR/DDR_DQ10: track 0.00 -> 20.3 mm
- net /DDR/DDR_DQ13: track 0.00 -> 18.2 mm
- net /DDR/DDR_DQ14: track 28.5 -> 17.8 mm
- net /DDR/DDR_DQS0_N: track 33.1 -> 22.6 mm, vias 0 -> 2
- net /DDR/DDR_DQS0_P: track 33.0 -> 22.8 mm, vias 0 -> 2
- net /DDR/DDR_DQ15: track 29.8 -> 23.6 mm
- net /DDR/DDR_DQ11: track 26.1 -> 21.1 mm
- net /DDR/DDR_DQ12: track 27.4 -> 23.0 mm
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Other:
- copper layers 2 -> 6

Commit message: PCB_UPDATE
Connections:
- U401 pad B8: /DDR/DDR_DQ4 -> /DDR/DDR_DQ5
- U401 pad C8: /DDR/DDR_DQ5 -> /DDR/DDR_DQ4
Routing:
- net /DDR/DDR_DQ5: track 0.00 -> 24.2 mm, vias 0 -> 2
- net /DDR/DDR_DQ2: track 0.00 -> 23.7 mm, vias 0 -> 2
- net /DDR/DDR_DQ4: track 0.00 -> 22.5 mm, vias 0 -> 2
- net /DDR/DDR_DQM1: track 0.00 -> 20.8 mm
- net /DDR/DDR_DQM0: track 0.00 -> 20.7 mm, vias 0 -> 2
- net /DDR/DDR_DQ6: track 0.00 -> 20.2 mm, vias 0 -> 2
- net /DDR/DDR_CLK_P: track 0.00 -> 14.9 mm, vias 0 -> 2
- net /DDR/DDR_CLK_N: track 0.00 -> 14.7 mm, vias 0 -> 2
- net /DDR/DDR_A10: track 0.00 -> 12.6 mm, vias 0 -> 2
- net /DDR/DDR_A1: track 0.00 -> 12.2 mm, vias 0 -> 2
- net /DDR/DDR_A4: track 0.00 -> 11.9 mm, vias 0 -> 2
- net /DDR/DDR_A8: track 0.00 -> 11.1 mm, vias 0 -> 2
- net /DDR/DDR_A0: track 1.47 -> 11.9 mm, vias 0 -> 2
- net /DDR/DDR_A11: track 0.00 -> 10.4 mm, vias 0 -> 2
- net /DDR/DDR_A14: track 0.00 -> 9.54 mm, vias 0 -> 2
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
Commit message: pcb_update
Parts:
- added R430: 56, Resistor_SMD:R_0402_1005Metric, B.Cu at (105.8, 75.0)
- R407, R410, R412, R414, R416, R417, R418, R420, R422, R426: moved to B.Cu
- moved C410 67.6 mm to (88.7, 93.3)
- moved C411 67.6 mm to (88.7, 95.3)
- moved C412 67.6 mm to (88.7, 97.2)
- moved C418 67.6 mm to (91.6, 93.3)
- moved C407 67.6 mm to (85.8, 103.1)
- moved C408 67.6 mm to (85.8, 105.1)
- moved C413 67.6 mm to (88.7, 99.2)
- moved C414 67.6 mm to (88.7, 101.2)
- moved C415 67.6 mm to (88.7, 103.1)
- moved C416 67.6 mm to (88.7, 105.1)
- moved C417 67.6 mm to (91.6, 91.3)
- moved C409 67.6 mm to (88.7, 91.3)
- moved R417 52.0 mm to (101.8, 75.0), turned to -90 degrees
- moved R418 50.4 mm to (104.8, 75.0), turned to -90 degrees
- moved R410 49.9 mm to (96.9, 75.0), turned to -90 degrees
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Connections:
- U301 pad L16: unconnected-(U301B-DDR_A15-PadL16) -> /DDR/DDR_A15
- U401 pad M7: unconnected-(U401-NC__4-PadM7) -> /DDR/DDR_A15
Routing:
- net /DDR/DDR_A15: track 0.00 -> 24.4 mm, vias 0 -> 2
- net /DDR/DDR_A12: track 0.00 -> 21.7 mm, vias 0 -> 2
- net /DDR/DDR_BA1: track 0.00 -> 16.7 mm, vias 0 -> 2
- net /DDR/DDR_CKE: track 0.00 -> 16.7 mm, vias 0 -> 2
- net /DDR/DDR_A6: track 0.00 -> 16.6 mm, vias 0 -> 2
- net /DDR/DDR_RASN: track 0.00 -> 16.3 mm, vias 0 -> 2
- net /DDR/DDR_WEN: track 0.00 -> 16.2 mm, vias 0 -> 2
- net /DDR/DDR_CASN: track 0.00 -> 15.9 mm, vias 0 -> 2
- net /DDR/DDR_BA2: track 0.00 -> 15.8 mm, vias 0 -> 2
- net /DDR/DDR_CSN: track 0.00 -> 15.8 mm, vias 0 -> 2
- net /DDR/DDR_ODT: track 0.00 -> 14.5 mm, vias 0 -> 2
- net /DDR/DDR_A9: track 0.00 -> 13.4 mm, vias 0 -> 2
- net /DDR/DDR_A2: track 0.00 -> 12.8 mm, vias 0 -> 2
- net /DDR/DDR_A13: track 0.00 -> 10.7 mm, vias 0 -> 2
- net /DDR/DDR_A14: track 9.54 -> 19.3 mm
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