File: PCB/MPU_MOD.kicad_pcb (KiCad board)
At the start: 6 copper layers, 50 x 50 mm, 295 parts, among them J501 MEM2090-00-145-00-A_REVA, J701 FTSH-107-01-L-DV-K-A, J801 USB4215-03-A_REVA, J901 73412-0110, U201 STC3115IQT, U202 BQ25606RGER, U203 STPMIC1APQR, U301 STM32MP157FABx, U401 MT41K256M16TW-107_P, U501 EMMC04G-W627-M06U, U502 HSP051-4M10, U503 HSP051-4M10, U701 HSP051-4M10, U702 HSP051-4M10, U801 FUSB302BMPX, U802 HSP051-4M10, U901 LBEE5PK2AE-771, Y601 NX2012SA-32.768K, Y701 ECS-2520MVQ-240

Commit message: PCB_UPDATE
Parts:
- moved R420 3.50 mm to (97.3, 75.0)
- moved R422 2.28 mm to (100.2, 75.0)
- moved R407 1.63 mm to (102.2, 75.0)
- moved R414 1.55 mm to (94.4, 75.0)
- moved R418 0.65 mm to (104.2, 75.0)
- moved R430 0.65 mm to (105.2, 75.0)
- moved R426 0.65 mm to (99.2, 75.0)
- moved R417 0.63 mm to (101.2, 75.0)
- moved R404 0.62 mm to (98.3, 74.0)
- moved R410 0.58 mm to (96.3, 75.0)
- moved R412 0.44 mm to (95.4, 75.0)
- moved R416 0.38 mm to (103.2, 75.0)
Routing:
- net /DDR/DDR_RASN: track 16.3 -> 0.00 mm, vias 2 -> 0
- net /DDR/DDR_WEN: track 16.2 -> 0.00 mm, vias 2 -> 0
- net /DDR/DDR_CASN: track 15.9 -> 0.00 mm, vias 2 -> 0
- net /DDR/DDR_BA2: track 15.8 -> 0.00 mm, vias 2 -> 0
- net /DDR/DDR_CSN: track 15.8 -> 0.00 mm, vias 2 -> 0
- net /DDR/DDR_ODT: track 14.5 -> 0.00 mm, vias 2 -> 0
- net /DDR/DDR_A9: track 13.4 -> 0.00 mm, vias 2 -> 0
- net /DDR/DDR_A0: track 13.1 -> 0.00 mm, vias 2 -> 0
- net /DDR/DDR_A2: track 12.8 -> 0.00 mm, vias 2 -> 0
- net /DDR/DDR_A13: track 10.7 -> 0.00 mm, vias 2 -> 0
- net /DDR/DDR_A15: track 24.4 -> 14.3 mm
- net /DDR/DDR_A12: track 21.7 -> 12.6 mm
- net /DDR/DDR_A11: track 20.0 -> 11.1 mm
- net /DDR/DDR_A14: track 19.3 -> 10.8 mm
- net /DDR/DDR_A1: track 21.9 -> 13.8 mm
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
Commit message: PCB_UPDATE
Parts:
- J501: moved to B.Cu
- moved J801 103.2 mm to (96.8, 105.3)
- moved U501 98.9 mm to (78.8, 86.8)
- moved U901 98.8 mm to (75.8, 101.4)
- moved J501 53.6 mm to (110.6, 100.6), turned to 180 degrees
- moved U203 34.2 mm to (105.2, 92.7)
- moved U202 32.2 mm to (114.6, 94.4)
- moved C401 16.7 mm to (98.3, 85.4)
- moved R401 16.7 mm to (100.4, 85.4)
Routing:
- net /DDR/DDR_DQS0_P: track 21.7 -> 26.0 mm
- net /DDR/DDR_DQS0_N: track 22.5 -> 26.6 mm
- net /DDR/DDR_DQ6: track 20.2 -> 23.9 mm
- net /DDR/DDR_DQ4: track 23.1 -> 24.3 mm
- net /DDR/DDR_DQ2: track 23.8 -> 24.4 mm

Commit message: PCB_UPDATE
Parts:
- R406, R408, R409, R411, R413, R415, R419, R421, R423, R424, R425, R427, R428, R429: moved to B.Cu
- moved C224 119.1 mm to (41.6, 123.5)
- moved C225 118.6 mm to (41.6, 124.4)
- moved C217 116.1 mm to (41.6, 122.6)
- moved C220 115.5 mm to (41.2, 126.4)
- moved C219 113.4 mm to (41.6, 120.8)
- moved C221 112.1 mm to (41.6, 121.7)
- moved C216 110.2 mm to (41.6, 125.3)
- moved C230 109.7 mm to (43.9, 129.7)
- moved R603 108.5 mm to (82.5, 80.3)
- moved R604 108.5 mm to (82.5, 82.3)
- moved C229 107.5 mm to (48.2, 129.7)
- moved C218 106.3 mm to (51.9, 122.8), turned to 180 degrees
- moved C228 106.2 mm to (41.8, 114.1)
- moved C226 106.1 mm to (52.5, 120.3), turned to 180 degrees
- moved C214 105.7 mm to (43.1, 127.4), turned to 90 degrees
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Routing:
- net /DDR/DDR_RASN: track 0.00 -> 24.9 mm, vias 0 -> 2
- net /DDR/DDR_BA2: track 0.00 -> 15.6 mm, vias 0 -> 2
- net /DDR/DDR_CSN: track 0.00 -> 15.3 mm, vias 0 -> 2
- net /DDR/DDR_WEN: track 0.00 -> 15.3 mm, vias 0 -> 2
- net /DDR/DDR_CASN: track 0.00 -> 15.1 mm, vias 0 -> 2
- net /DDR/DDR_ODT: track 0.00 -> 14.1 mm, vias 0 -> 2
- net /DDR/DDR_BA0: track 0.57 -> 13.7 mm, vias 1 -> 2

Commit message: PCB_UPDATE
Parts:
- added R514: 47k, Resistor_SMD:R_0402_1005Metric, F.Cu at (123.3, 155.8)
- added R515: 47k, Resistor_SMD:R_0402_1005Metric, F.Cu at (123.3, 157.8)
- added R516: 47k, Resistor_SMD:R_0402_1005Metric, F.Cu at (123.3, 159.8)
- added R517: 47k, Resistor_SMD:R_0402_1005Metric, F.Cu at (123.3, 161.8)
- added R518: 47k, Resistor_SMD:R_0402_1005Metric, F.Cu at (123.3, 163.8)
- added R519: 47k, Resistor_SMD:R_0402_1005Metric, F.Cu at (123.3, 165.8)
- C501, C502, C503, C504, C505, C506, C507, R509: moved to B.Cu
- moved R501 121.9 mm to (56.8, 47.4)
- moved R502 121.9 mm to (56.8, 49.4)
- moved R503 121.9 mm to (56.8, 51.4)
- moved R504 121.9 mm to (56.8, 53.4)
- moved R505 121.9 mm to (56.8, 55.4)
- moved R506 121.9 mm to (59.7, 47.4)
- moved R507 121.9 mm to (59.7, 49.4)
- moved R508 121.9 mm to (59.7, 51.4)
- moved R510 121.9 mm to (59.7, 55.4)
- moved R511 121.9 mm to (62.6, 47.4)
- moved R512 121.9 mm to (62.6, 49.4)
- moved C507 101.1 mm to (80.6, 47.9)
- moved C505 100.6 mm to (77.9, 51.3)
- moved C504 100.3 mm to (78.8, 47.9)
- moved R509 99.9 mm to (81.7, 56.6), turned to 180 degrees
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Connections:
- net SYS_I2C_SCL renamed SYS_I2C4_SCL
- net SYS_I2C_SDA renamed SYS_I2C4_SDA
- TP905 pad 1: I2S3_SDO -> I2S1_SDO
- TP906 pad 1: I2S3_WS -> I2S1_WS
- TP907 pad 1: I2S3_CK -> I2S1_CK
- TP908 pad 1: I2S3_SDI -> I2S1_SDI
- U301 pad A2: unconnected-(U301D-PG15-PadA2) -> SDMMC3_CK
- U301 pad A3: unconnected-(U301C-PD0-PadA3) -> SDMMC3_CMD
- U301 pad A4: unconnected-(U301C-PD1-PadA4) -> SDMMC3_D0
- U301 pad B1: unconnected-(U301D-PE1-PadB1) -> UART8_TX_STM
- U301 pad B4: unconnected-(U301C-PD7-PadB4) -> SDMMC3_D3
- U301 pad C4: unconnected-(U301D-PE0-PadC4) -> UART8_RX_STM
- U301 pad D3: unconnected-(U301D-PE14-PadD3) -> UART8_RTS_STM
- U301 pad D6: unconnected-(U301C-PD4-PadD6) -> SDMMC3_D1
- U301 pad D7: unconnected-(U301C-PD5-PadD7) -> SDMMC3_D2
- U301 pad E1: unconnected-(U301D-PE15-PadE1) -> UART8_CTS_STM
- U301 pad P4: unconnected-(U301C-PA5-PadP4) -> I2S1_CK
- U301 pad R4: unconnected-(U301C-PA4-PadR4) -> I2S1_WS
- U301 pad T2: unconnected-(U301C-PC2-PadT2) -> I2S1_SDI
- U301 pad T5: unconnected-(U301C-PA6-PadT5) -> I2S1_SDI
- U301 pad T6: unconnected-(U301C-PA7-PadT6) -> I2S1_SDO
- U301 pad V2: unconnected-(U301C-PC1-PadV2) -> I2S1_SDO
- U301 pad V5: unconnected-(U301C-PB12-PadV5) -> I2S1_WS
- U301 pad W5: unconnected-(U301C-PB10-PadW5) -> I2S1_CK
- U901 pad 6: I2S3_SDI -> I2S1_SDI
- U901 pad 7: I2S3_CK -> I2S1_CK
- U901 pad 8: I2S3_WS -> I2S1_WS
- U901 pad 9: I2S3_SDO -> I2S1_SDO
Other:
- board size 50 x 50 mm -> 47 x 100 mm

Commit message: PCD_UPDATE
Parts:
- removed C501: 2.2uF, Capacitor_SMD:C_0402_1005Metric
- removed U501: EMMC04G-W627-M06U, lib:BGA153N50P14X14_1300X1150X100N
- added C509: 1uF, Capacitor_SMD:C_0402_1005Metric, B.Cu at (76.8, 45.4)
- added C510: 100nF, Capacitor_SMD:C_0402_1005Metric, B.Cu at (83.9, 48.0)
- added C511: 100nF, Capacitor_SMD:C_0402_1005Metric, B.Cu at (75.8, 48.4)
- added C512: 100nF, Capacitor_SMD:C_0402_1005Metric, B.Cu at (81.9, 48.3)
- added C513: 100nF, Capacitor_SMD:C_0402_1005Metric, B.Cu at (81.5, 55.9)
- added C514: 100nF, Capacitor_SMD:C_0402_1005Metric, B.Cu at (76.3, 56.0)
- added U1: IS21ES08GA-JQLI-TR, lib:FBGA100_ISI, F.Cu at (78.9, 50.3)
- R501, R502, R503, R504, R505, R506, R507, R508, R510, R511, R512: moved to B.Cu
- moved R505 28.3 mm to (85.0, 54.3), turned to -90 degrees
- moved R503 28.2 mm to (85.0, 52.1), turned to 90 degrees
- moved R502 27.8 mm to (84.0, 54.8), turned to -90 degrees
- moved R504 27.3 mm to (84.0, 52.7), turned to 90 degrees
- moved R501 24.7 mm to (79.4, 57.6), turned to -90 degrees
- moved R511 14.2 mm to (76.1, 43.0), turned to 180 degrees
- moved R506 14.2 mm to (73.2, 43.0), turned to 180 degrees
- moved R507 14.2 mm to (73.2, 45.0), turned to 180 degrees
- moved R508 14.2 mm to (73.2, 47.0), turned to 180 degrees
- moved R512 14.0 mm to (73.5, 58.2), turned to 90 degrees
- moved R510 13.1 mm to (72.5, 58.2), turned to -90 degrees
- moved R509 11.9 mm to (73.2, 48.3), turned to 0 degrees
- moved C502 7.82 mm to (76.8, 47.3), turned to 90 degrees
- moved C507 5.44 mm to (80.9, 53.3), turned to -90 degrees
- moved C504 5.42 mm to (76.3, 52.7), turned to 180 degrees
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Routing:
- net SDMMC2_D7: track 0.00 -> 15.5 mm, vias 0 -> 2
- net SDMMC2_D5: track 0.00 -> 14.0 mm, vias 0 -> 2
- net SDMMC2_D0: track 0.00 -> 13.7 mm, vias 0 -> 2
- net SDMMC2_D2: track 0.00 -> 13.2 mm, vias 0 -> 2
- net SDMMC2_D6: track 0.00 -> 13.1 mm, vias 0 -> 2
- net SDMMC2_D4: track 0.00 -> 9.81 mm, vias 0 -> 2
- net SDMMC2_D3: track 0.00 -> 9.44 mm, vias 0 -> 2
- net SDMMC2_NRST: track 0.00 -> 8.88 mm, vias 0 -> 1
- net SDMMC2_D1: track 0.00 -> 8.72 mm, vias 0 -> 2
- net SDMMC2_CK: track 0.00 -> 5.30 mm, vias 0 -> 1
- net Net-(U1-CLK): track 0.00 -> 1.72 mm, vias 0 -> 1
Other:
- copper layers 6 -> 8

Commit message: PCB_UPDATE
Parts:
- removed C801: 100nF, Capacitor_SMD:C_0402_1005Metric
- added C515: 1uF, Capacitor_SMD:C_0402_1005Metric, F.Cu at (93.8, 78.6)
- added Q1: STL9P3LLH6, lib:TRANS_STL9P3LLH6, F.Cu at (66.2, 88.6)
- added U3: BQ24298RTWR, lib:BQ24298, F.Cu at (77.3, 92.8)
- moved C508 124.1 mm to (116.3, 46.0), turned to 90 degrees
- moved R513 116.3 mm to (109.3, 47.1), turned to 90 degrees
- moved J501 115.9 mm to (113.5, 51.3), turned to -90 degrees
- moved C805 113.3 mm to (83.6, 86.7), turned to 90 degrees
- moved U502 112.9 mm to (109.2, 50.2), turned to 90 degrees
- moved U503 109.5 mm to (109.3, 53.6), turned to 90 degrees
- moved C803 108.9 mm to (83.0, 84.1), turned to 90 degrees
- moved D801 108.0 mm to (86.7, 81.9), turned to 180 degrees
- moved U802 107.7 mm to (89.4, 81.8)
- moved C804 107.4 mm to (84.0, 84.1), turned to -90 degrees
- moved U801 104.8 mm to (93.0, 81.1), turned to 180 degrees
- moved TP802 101.8 mm to (84.9, 94.6)
- moved U901 99.4 mm to (91.8, 49.0)
- moved C802 96.2 mm to (95.3, 79.2), turned to -90 degrees
- moved C228 77.7 mm to (111.5, 79.8), turned to -90 degrees
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Connections:
- C802 pad 2: Net-(C801-Pad2) -> VDD
- U801 pad 3: Net-(C801-Pad2) -> VDD
- U801 pad 4: Net-(C801-Pad2) -> VDD
- U802 pad 1: USB_D- -> USB_CC1
- U802 pad 10: USB_D- -> USB_CC1
- U802 pad 2: USB_D+ -> USB_D-
- U802 pad 4: USB_CC2 -> USB_D+
- U802 pad 5: USB_CC1 -> USB_CC2
- U802 pad 6: USB_CC1 -> USB_CC2
- U802 pad 7: USB_CC2 -> USB_D+
- U802 pad 9: USB_D+ -> USB_D-
Other:
- board size 47 x 100 mm -> 45 x 50 mm

Commit message: PCB_UPDATE
Parts:
- removed C201, C202, C203, C208, C209: 10uF, Capacitor_SMD:C_0603_1608Metric
- removed C206: 47nF, Capacitor_SMD:C_0402_1005Metric
- removed C207: 4.7uF, Capacitor_SMD:C_0402_1005Metric
- removed D201: LED_R, LED_SMD:LED_0402_1005Metric
- removed D202: LED_B, LED_SMD:LED_0402_1005Metric
- removed L201: 1uH, Inductor_SMD:L_1008_2520Metric
- removed Q1: STL9P3LLH6, lib:TRANS_STL9P3LLH6
- removed R203, R207: 0, Resistor_SMD:R_0402_1005Metric
- removed R204, R205: 2k2, Resistor_SMD:R_0402_1005Metric
- removed R206: 220, Resistor_SMD:R_0402_1005Metric
- removed R208: 10k, Resistor_SMD:R_0402_1005Metric
- removed R211: 240, Resistor_SMD:R_0402_1005Metric
- removed R213: 5k23, Resistor_SMD:R_0402_1005Metric
- removed R214: 30k1, Resistor_SMD:R_0402_1005Metric
- removed U202: BQ25606RGER, lib:QFN50P400X400X100-25N
- added C232: 47nF, Capacitor_SMD:C_0402_1005Metric, F.Cu at (83.5, 82.8)
- added C233: 10uF, Capacitor_SMD:C_0603_1608Metric, F.Cu at (80.9, 86.8)
- added C234: 10uF, Capacitor_SMD:C_0603_1608Metric, F.Cu at (81.0, 85.1)
- added C235: 4.7uF, Capacitor_SMD:C_0402_1005Metric, F.Cu at (83.5, 81.5)
- added C236: 10uF, Capacitor_SMD:C_0603_1608Metric, F.Cu at (78.0, 85.1)
- added C237: 1uF, Capacitor_SMD:C_0402_1005Metric, F.Cu at (81.9, 79.0)
- added C238: 8.2uF, Capacitor_SMD:C_0402_1005Metric, F.Cu at (83.5, 80.6)
- added D1: LED, LED_SMD:LED_0402_1005Metric, F.Cu at (69.3, 77.2)
- added D2: LED, LED_SMD:LED_0402_1005Metric, F.Cu at (69.3, 79.1)
- added J1: SJ3-35024K-SMT-TR, lib:SAMESKY_SJ3-35024K-SMT-TR, F.Cu at (112.0, 98.3)
- added J2: 2-1734248-0, lib:CONN_2-1734248-0_TYCO, F.Cu at (100.9, 37.1)
- added L206: 1uH, Inductor_SMD:L_1008_2520Metric, F.Cu at (84.1, 85.3)
- added R216: 5k25, Resistor_SMD:R_0402_1005Metric, F.Cu at (76.8, 83.9)
- added R217: 31k23, Resistor_SMD:R_0402_1005Metric, F.Cu at (76.8, 83.0)
- added R218: 317, Resistor_SMD:R_0402_1005Metric, F.Cu at (76.8, 82.0)
- added R219: 10k, Resistor_SMD:R_0402_1005Metric, F.Cu at (76.8, 80.7)
- added R220: 1k, Resistor_SMD:R_0402_1005Metric, F.Cu at (70.3, 79.1)
- added R221: 1k, Resistor_SMD:R_0402_1005Metric, F.Cu at (70.3, 77.2)
- C403, C421, C422, C423, C428, C429: moved to F.Cu
- C407, C408, C409, C410, C411, C412, C413, C414, C415, C416, C417, C418: moved to B.Cu
- TP201, TP202, TP203, TP204, TP205, TP206, TP207, TP208, TP209, TP210, TP211, TP212, TP401, TP402, TP403, TP601, TP602, TP701, TP702, TP703, TP704, TP705, TP706, TP707, TP708, TP709, TP710, TP801, TP802, TP803, TP804, TP805, TP806, TP901, TP902, TP903, TP904, TP905, TP906, TP907, TP908: footprint TestPoint:TestPoint_Pad_D1.0mm -> Library:TP_0.5mm
- moved S605 140.4 mm to (70.0, 38.4), turned to -90 degrees
- moved S602 135.3 mm to (69.9, 32.4), turned to -90 degrees
- moved S604 134.2 mm to (70.0, 44.4), turned to -90 degrees
- moved C602 132.1 mm to (70.0, 63.7), turned to 180 degrees
- moved C601 130.8 mm to (70.0, 64.9)
- moved S603 128.6 mm to (70.0, 50.4), turned to -90 degrees
- moved Y601 127.4 mm to (71.8, 64.2), turned to -90 degrees
- moved D602 127.0 mm to (69.3, 75.2), turned to -90 degrees
- moved D601 126.9 mm to (69.3, 73.3), turned to -90 degrees
- moved R801 126.2 mm to (65.6, 69.0)
- moved S601 121.8 mm to (70.0, 56.5), turned to -90 degrees
- moved R602 121.1 mm to (70.3, 75.2), turned to 90 degrees
- moved R601 121.0 mm to (70.3, 73.3), turned to 90 degrees
- moved R514 112.8 mm to (108.3, 44.0)
- moved R515 112.8 mm to (108.3, 46.0)
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Connections:
- R201 pad 2: +BATT -> VDD
- R202 pad 2: +BATT -> VDD
- TP201 pad 1: CHRG_NPG -> Net-(U3-STAT)
- TP202 pad 1: CHRG_STAT -> Net-(U3-PG_N)
- U3 pad 1: unconnected-(U3-VBUS-Pad1) -> V_USB
- U3 pad 10: unconnected-(U3-ILIM-Pad10) -> Net-(U3-ILIM)
- U3 pad 11: unconnected-(U3-TS-Pad11) -> /PWR/BATT_T
- U3 pad 13: unconnected-(U3-BAT-Pad13) -> +BATT
- U3 pad 14: unconnected-(U3-BAT-Pad14) -> +BATT
- U3 pad 15: unconnected-(U3-SYS-Pad15) -> VIN
- U3 pad 16: unconnected-(U3-SYS-Pad16) -> VIN
- U3 pad 17: unconnected-(U3-PGND-Pad17) -> GND
- U3 pad 18: unconnected-(U3-PGND-Pad18) -> GND
- U3 pad 19: unconnected-(U3-SW-Pad19) -> Net-(C232-Pad1)
- U3 pad 2: unconnected-(U3-PSEL-Pad2) -> CHRG_PSEL
- U3 pad 20: unconnected-(U3-SW-Pad20) -> Net-(C232-Pad1)
- U3 pad 21: unconnected-(U3-BTST-Pad21) -> Net-(U3-BTST)
- U3 pad 22: unconnected-(U3-REGN-Pad22) -> /PWR/REGN
- U3 pad 23: unconnected-(U3-PMID-Pad23) -> Net-(U3-PMID)
- U3 pad 24: unconnected-(U3-VBUS-Pad24) -> V_USB
- U3 pad 25: unconnected-(U3-PAD-Pad25) -> GND
- U3 pad 3: unconnected-(U3-PG_N-Pad3) -> Net-(U3-PG_N)
- U3 pad 4: unconnected-(U3-STAT-Pad4) -> Net-(U3-STAT)
- U3 pad 5: unconnected-(U3-SCL-Pad5) -> SYS_I2C4_SCL
- U3 pad 6: unconnected-(U3-SDA-Pad6) -> SYS_I2C4_SDA
- U3 pad 7: unconnected-(U3-INT-Pad7) -> CHRG_INT
- U3 pad 8: unconnected-(U3-OTG-Pad8) -> CHRG_OTG_ON
- U3 pad 9: unconnected-(U3-CE_N-Pad9) -> GND
Routing:
- net VIN: track 0.00 -> 14.4 mm, vias 0 -> 9
- net Net-(U203-LDO1OUT): track 0.00 -> 3.99 mm, vias 0 -> 1
- net Net-(U203-VLX3): track 0.00 -> 3.90 mm
- net Net-(U203-VLX1): track 0.00 -> 3.69 mm
- net 3V3: track 0.00 -> 3.09 mm, vias 0 -> 13
- net Net-(U203-VLX2): track 0.00 -> 2.94 mm
- net Net-(U203-LDO6OUT): track 0.00 -> 2.79 mm, vias 0 -> 1
- net VDD_DDR: track 0.00 -> 2.59 mm, vias 0 -> 8
- net VDDA: track 0.00 -> 2.28 mm, vias 0 -> 1
- net PWR_ON: track 0.00 -> 2.16 mm, vias 0 -> 1
- net VTT_DDR: track 0.00 -> 2.13 mm, vias 0 -> 2
- net Net-(U203-LDO2OUT): track 0.00 -> 2.06 mm, vias 0 -> 1
- net Net-(U203-VLX4): track 0.00 -> 2.05 mm
- net Net-(U203-~{RST}): track 0.00 -> 2.02 mm
- net VREF_DDR: track 0.00 -> 1.82 mm, vias 0 -> 1
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- added copper zone on F.Cu, net 3V3
- added copper zone on F.Cu, net GND
- added copper zone on F.Cu, net VDD
- added copper zone on F.Cu, net VDD_CORE
- added copper zone on F.Cu, net VDD_DDR
Other:
- board size 45 x 50 mm -> 45 x 70 mm
