File: PCB/MPU_MOD.kicad_pcb (KiCad board)
At the start: 8 copper layers, 45 x 70 mm, 305 parts, among them J1 SJ3-35024K-SMT-TR, J2 2-1734248-0, J501 MEM2090-00-145-00-A_REVA, J701 FTSH-107-01-L-DV-K-A, J801 USB4215-03-A_REVA, J901 73412-0110, U1 IS21ES08GA-JQLI-TR, U201 STC3115IQT, U203 STPMIC1APQR, U3 BQ24298RTWR, U301 STM32MP157FABx, U401 MT41K256M16TW-107_P, U502 HSP051-4M10, U503 HSP051-4M10, U701 HSP051-4M10, U702 HSP051-4M10, U801 FUSB302BMPX, U802 HSP051-4M10, U901 LBEE5PK2AE-771, Y601 NX2012SA-32.768K, Y701 ECS-2520MVQ-240

Commit message: PCB_UPDATE
Parts:
- C301, C302, C303, C304, C305, C306, C307, C308, C309, C310, C311, C312, C313, C314, C315, C316, C317, C318, C319, C320, C321, C322, C323, C324, C325, C326, C327, C328, C329, C330, C331, C333, C334, C335, C336, C337, C338, C339: moved to B.Cu
- L301: footprint Inductor_SMD:L_0201_0603Metric -> Inductor_SMD:L_0603_1608Metric
- moved C401 42.9 mm to (15.1, 91.9)
- moved R401 42.9 mm to (11.9, 91.2)
- moved R604 42.9 mm to (9.63, 94.8)
- moved R707 42.9 mm to (20.9, 91.1)
- moved R708 42.9 mm to (20.9, 93.1)
- moved R801 42.9 mm to (24.9, 82.7)
- moved C702 42.9 mm to (12.3, 87.2)
- moved R603 42.9 mm to (9.23, 93.0)
- moved R702 42.9 mm to (18.0, 93.1)
- moved R703 42.9 mm to (18.0, 95.1)
- moved R704 42.9 mm to (18.0, 97.1)
- moved R705 42.9 mm to (18.0, 99.1)
- moved C331 38.8 mm to (84.1, 65.6), turned to 45 degrees
- moved C335 35.5 mm to (85.7, 75.6), turned to 90 degrees
- moved C334 33.8 mm to (86.2, 62.4), turned to -90 degrees
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Routing:
- net GND: track 0.00 -> 62.2 mm, vias 46 -> 89
- net VDD_CORE: track 0.77 -> 56.4 mm, vias 8 -> 29
- net VDD: track 0.93 -> 15.0 mm, vias 11 -> 24
- net VDD_DDR: track 2.59 -> 8.78 mm, vias 8 -> 14
- net Net-(U301A-VREF+): track 0.00 -> 2.69 mm, vias 0 -> 1
- net Net-(U301A-VDDA): track 0.00 -> 2.16 mm, vias 0 -> 1
