File: PCB/HS_intrf.kicad_sch (KiCad schematic)
At the start: 13 parts, among them J3 USB4215-03-A_REVA, U11 HSP051-4M10, U2 STM32MP157FABx

Commit message: PCB_UPDATE
Parts:
- added C801, C802: 100nF, Capacitor_SMD:C_0402_1005Metric, symbol Device:C
- added TP801: TestPoint, TestPoint:TestPoint_Pad_D1.0mm, symbol Connector:TestPoint
- added U801: FUSB302BMPX, lib:MLP14_2P5X2P5_ONS, symbol FUSB302BMPX:FUSB302BMPX
- D801: renamed from D6; value SMAJ5.0A -> ESDA7P120-1U1M; footprint Diode_SMD:D_SMA -> lib:DIODE_ESDA7P120-1U1M_STM
- renumbered C105 to C803, C106 to C804, C107 to C805, J3 to J801, R62 to R801, TP32 to TP802, TP18 to TP803, TP19 to TP804, TP20 to TP805, TP21 to TP806, U2 to U301, U11 to U802
Connections:
- net GND: now also C801.1, C802.1, U801.15 (EPAD), U801.8 (GND), U801.9 (GND)
- net USB_CC1: now also U801.10 (CC1), U801.11 (CC1)
- net USB_CC2: now also U801.1 (CC2), U801.14 (CC2)
- net V_USB: now also U801.2 (VBUS)
- new net: C801.2, C802.2, U801.3 (VDD), U801.4 (VDD)
- new net: TP801.1, U801.12 (VCONN), U801.13 (VCONN)
- new net INT_USB_ctrl: U801.5 (INT_N)
- new net SYS_I2C_SCL: U801.6 (SCL)
- new net SYS_I2C_SDA: U801.7 (SDA)

Commit message: pcb_update
Connections:
- net SYS_I2C_SCL renamed SYS_I2C4_SCL
- net SYS_I2C_SDA renamed SYS_I2C4_SDA
Changed lines of the file:
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@@
 		)
 	)
-	(global_label "SYS_I2C_SDA"
+	(global_label "SYS_I2C4_SDA"
 		(shape input)
 		(at 62.23 167.64 180)
@@
 		)
 		(property "Intersheetrefs" "${INTERSHEET_REFS}"
-			(at 47.1496 167.64 0)
+			(at 45.9401 167.64 0)
 			(effects
 				(font
@@
 		)
 	)
-	(global_label "SYS_I2C_SCL"
+	(global_label "SYS_I2C4_SCL"
 		(shape input)
 		(at 62.23 165.1 180)
@@
 		)
 		(property "Intersheetrefs" "${INTERSHEET_REFS}"
-			(at 47.2101 165.1 0)
-			(effects
-				(font
+			(at 46.0006 165.1 0)
+			(effects
+				(font
