File: PCB/HS_intrf.kicad_sch (KiCad schematic)
At the start: 18 parts, among them J801 USB4215-03-A_REVA, Q1 STL9P3LLH6, U301 STM32MP157FABx, U801 FUSB302BMPX, U802 HSP051-4M10

Commit message: PCB_UPDATE
Parts:
- removed Q1: STL9P3LLH6, lib:TRANS_STL9P3LLH6, symbol STL9P3LLH6:STL9P3LLH6
- added J2: 2-1734248-0, lib:CONN_2-1734248-0_TYCO, symbol 2-1734248-0:2-1734248-0
- TP801, TP802, TP803, TP804, TP805, TP806: footprint TestPoint:TestPoint_Pad_D1.0mm -> Library:TP_0.5mm
Connections:
- no-connect marks 0 -> 20
Changed lines of the file:
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@@
 		(color 0 0 0 0)
 	)
+	(no_connect
+		(at 36.83 97.79)
+	)
+	(no_connect
+		(at 36.83 77.47)
+	)
+	(no_connect
+		(at 36.83 100.33)
+	)
+	(no_connect
+		(at 36.83 72.39)
+	)
+	(no_connect
+		(at 36.83 87.63)
+	)
+	(no_connect
+		(at 36.83 95.25)
+	)
+	(no_connect
+		(at 36.83 110.49)
+	)
+	(no_connect
+		(at 36.83 105.41)
+	)
+	(no_connect
+		(at 36.83 74.93)
+	)
+	(no_connect
+		(at 36.83 92.71)
+	)
+	(no_connect
+		(at 36.83 115.57)
+	)
+	(no_connect
+		(at 36.83 102.87)
+	)
+	(no_connect
+		(at 36.83 82.55)
+	)
+	(no_connect
+		(at 36.83 85.09)
+	)
+	(no_connect
+		(at 36.83 113.03)
+	)
+	(no_connect
+		(at 36.83 90.17)
+	)
+	(no_connect
+		(at 36.83 69.85)
+	)
+	(no_connect
+		(at 36.83 80.01)
+	)
+	(no_connect
+		(at 36.83 118.11)
+	)
+	(no_connect
+		(at 36.83 107.95)
+	)
 	(wire
 		(pts
@@
 			)
 		)
-		(property "Footprint" "TestPoint:TestPoint_Pad_D1.0mm"
+		(property "Footprint" "Library:TP_0.5mm"
 			(at 248.92 43.18 0)
 			(effects
@@
 			)
 		)
-		(property "Footprint" "TestPoint:TestPoint_Pad_D1.0mm"
+		(property "Footprint" "Library:TP_0.5mm"
 			(at 213.36 27.94 0)
 			(effects
@@
 			)
 		)
-		(property "Footprint" "TestPoint:TestPoint_Pad_D1.0mm"
+		(property "Footprint" "Library:TP_0.5mm"
 			(at 233.68 43.18 0)
 			(effects
@@
 			)
 		)
-		(property "Footprint" "TestPoint:TestPoint_Pad_D1.0mm"
+		(property "Footprint" "Library:TP_0.5mm"
 			(at 241.3 43.18 0)
 			(effects
@@
 	)
 	(symbol
+		(lib_id "2-1734248-0:2-1734248-0")
+		(at 36.83 19.05 0)
+		(mirror y)
+		(unit 1)
+		(exclude_from_sim no)
+		(in_bom yes)
+		(on_board yes)
+		(dnp no)
+		(property "Reference" "J2"
+			(at 22.86 67.3099 0)
+			(effects
+				(font
+					(size 1.524 1.524)
+				)
+				(justify left)
+			)
+		)
+		(property "Value" "2-1734248-0"
+			(at 22.86 69.8499 0)
+			(effects
+				(font
+					(size 1.524 1.524)
+				)
+				(justify left)
+			)
+		)
+		(property "Footprint" "lib:CONN_2-1734248-0_TYCO"
+			(at 36.83 19.05 0)
+			(effects
+				(font
+					(size 1.27 1.27)
+					(italic yes)
+				)
+				(hide yes)
+			)
+		)
+		(property "Datasheet" "2-1734248-0"
+			(at 36.83 19.05 0)
+			(effects
+				(font
+					(size 1.27 1.27)
+					(italic yes)
+				)
+				(hide yes)
+			)
+		)
+		(property "Description" ""
+			(at 36.83 19.05 0)
+			(effects
+				(font
+					(size 1.27 1.27)
+				)
+				(hide yes)
+			)
+		)
+		(pin "11"
+		)
+		(pin "17"
+		)
+		(pin "12"
+		)
+		(pin "10"
+		)
+		(pin "6"
+		)
+		(pin "34"
+		)
+		(pin "30"
+		)
+		(pin "9"
+		)
+		(pin "25"
+		)
+		(pin "4"
+		)
+		(pin "7"
+		)
+		(pin "31"
+		)
+		(pin "3"
+		)
+		(pin "38"
+		)
+		(pin "20"
+		)
+		(pin "13"
+		)
+		(pin "27"
+		)
+		(pin "21"
+		)
+		(pin "18"
+		)
+		(pin "29"
+		)
+		(pin "32"
+		)
+		(pin "8"
+		)
+		(pin "14"
+		)
+		(pin "15"
+		)
+		(pin "22"
+		)
+		(pin "24"
+		)
+		(pin "23"
+		)
+		(pin "35"
+		)
+		(pin "37"
+		)
+		(pin "1"
+		)
+		(pin "16"
+		)
+		(pin "40"
+		)
+		(pin "19"
+		)
+		(pin "39"
+		)
+		(pin "2"
+		)
+		(pin "5"
+		)
+		(pin "28"
+		)
+		(pin "36"
+		)
+		(pin "33"
+		)
+		(pin "26"
+		)
+		(instances
+			(project ""
+				(path "/65890f61-d586-475b-928a-b635a5e4e59e/9899e005-10ba-4bf4-b936-8d0d8a1813b9"
+					(reference "J2")
+					(unit 1)
+				)
+			)
+		)
+	)
+	(symbol
 		(lib_id "Device:R")
 		(at 78.74 83.82 180)
@@
 			)
 		)
-		(property "Footprint" "TestPoint:TestPoint_Pad_D1.0mm"
+		(property "Footprint" "Library:TP_0.5mm"
 			(at 226.06 43.18 0)
 			(effects
@@
 			)
 		)
-		(property "Footprint" "TestPoint:TestPoint_Pad_D1.0mm"
+		(property "Footprint" "Library:TP_0.5mm"
 			(at 59.69 154.94 0)
 			(effects
@@
 					(unit 1)
 				)
-			)
-		)
-	)
-	(symbol
-		(lib_id "STL9P3LLH6:STL9P3LLH6")
-		(at 48.26 124.46 0)
-		(unit 1)
-		(exclude_from_sim no)
-		(in_bom yes)
-		(on_board yes)
-		(dnp no)
-		(fields_autoplaced yes)
-		(property "Reference" "Q1"
-			(at 53.34 123.1899 0)
-			(effects
-				(font
-					(size 1.27 1.27)
-				)
-				(justify left)
-			)
-		)
-		(property "Value" "STL9P3LLH6"
-			(at 53.34 125.7299 0)
-			(effects
-				(font
-					(size 1.27 1.27)
-				)
-				(justify left)
-			)
-		)
-		(property "Footprint" "lib:TRANS_STL9P3LLH6"
-			(at 48.26 124.46 0)
-			(effects
-				(font
-					(size 1.27 1.27)
-				)
-				(justify bottom)
-				(hide yes)
-			)
-		)
-		(property "Datasheet" ""
-			(at 48.26 124.46 0)
-			(effects
-				(font
-					(size 1.27 1.27)
-				)
-				(hide yes)
-			)
-		)
-		(property "Description" ""
-			(at 48.26 124.46 0)
-			(effects
-				(font
-					(size 1.27 1.27)
-				)
-				(hide yes)
-			)
-		)
-		(property "PARTREV" "3"
-			(at 48.26 124.46 0)
-			(effects
-				(font
-					(size 1.27 1.27)
-				)
-				(justify bottom)
-				(hide yes)
-			)
-		)
-		(property "MANUFACTURER" "ST Microelectronics"
-			(at 48.26 124.46 0)
-			(effects
-				(font
-					(size 1.27 1.27)
-				)
-				(justify bottom)
-				(hide yes)
-			)
-		)
-		(property "MAXIMUM_PACKAGE_HEIGHT" "0.9mm"
-			(at 48.26 124.46 0)
-			(effects
-				(font
-					(size 1.27 1.27)
-				)
-				(justify bottom)
-				(hide yes)
-			)
-		)
-		(property "STANDARD" "Manufacturer recommendations"
-			(at 48.26 124.46 0)
-			(effects
-				(font
-					(size 1.27 1.27)
-				)
-				(justify bottom)
-				(hide yes)
-			)
-		)
-		(pin "4"
-		)
-		(pin "5_1"
-		)
-		(pin "1"
-		)
-		(pin "5"
-		)
-		(pin "2"
-		)
-		(pin "3"
-		)
-		(pin "5_2"
-		)
-		(instances
-			(project ""
-				(path "/65890f61-d586-475b-928a-b635a5e4e59e/9899e005-10ba-4bf4-b936-8d0d8a1813b9"
-					(reference "Q1")
-					(unit 1)
-				)
