File: PCB/FLASH_SD.kicad_sch (KiCad schematic)
At the start: 36 parts, among them J501 MEM2090-00-145-00-A_REVA, U1 IS21ES08GA-JQLI-TR, U502 HSP051-4M10, U503 HSP051-4M10

Commit message: PCB_UPDATE
Parts:
- U1: footprint FBGA100_ISI -> lib:FBGA100_ISI
