File: PCB/IO_Perph_Conn.kicad_sch (KiCad schematic)
At the start: 16 parts, among them U2 STM32MP157FABx, Y2 NX2012SA-32.768K

Commit message: PCB_UPDATE
Parts:
- removed C116: 10nF, Capacitor_SMD:C_0402_1005Metric, symbol Device:C
- removed D8: PTVS3V3S1UR, PTVS3V3S1UR:TVS_PTVS3V3S1UR, symbol PTVS3V3S1UR:PTVS3V3S1UR
- removed R63: 10k, Resistor_SMD:R_0402_1005Metric, symbol Device:R
- removed S4: PTS525SM15SMTR2LFS, lib:SW_PTS525SM15SMTR2LFS, symbol PTS525SM15SMTR2LFS:PTS525SM15SMTR2LFS
- added S601, S602, S603, S604, S605: EVQ-9P701P, lib:SW_EVQ-9P701P, symbol EVQ-9P701P:EVQ-9P701P
- renumbered C114 to C601, C115 to C602, D3 to D601, D2 to D602, R43 to R601, R44 to R602, R60 to R603, R61 to R604, TP15 to TP601, TP14 to TP602, U2 to U301, Y2 to Y601
Connections:
- net EXT_WKUP renamed PWR_SW_WAKE_UP

Commit message: pcb_update
Connections:
- net UART8_CTS_STM: now also U301.E1 (PE15)
- net UART8_RTS_STM: now also U301.D3 (PE14)
- net UART8_RX_STM: now also U301.C4 (PE0)
- net UART8_TX_STM: now also U301.B1 (PE1)
- net SDMMC3_CK: now reaches U301.A2 (PG15)
- net SDMMC3_CMD: now reaches U301.A3 (PD0)
- net SDMMC3_D0: now reaches U301.A4 (PD1)
- net SDMMC3_D3: now reaches U301.B4 (PD7)
- net SDMMC3_D1: now reaches U301.D6 (PD4)
- net SDMMC3_D2: now reaches U301.D7 (PD5)
- net I2S1_CK: now reaches U301.P4 (PA5)
- net I2S1_CK: now also U301.W5 (PB10)
- net I2S1_WS: now reaches U301.R4 (PA4)
- net I2S1_WS: now also U301.V5 (PB12)
- net I2S1_SDI: now reaches U301.T2 (PC2)
- net I2S1_SDI: now also U301.T5 (PA6)
- net I2S1_SDO: now reaches U301.T6 (PA7)
- net I2S1_SDO: now also U301.V2 (PC1)
- net SYS_I2C_SCL renamed SYS_I2C4_SCL
- net SYS_I2C_SDA renamed SYS_I2C4_SDA
Other:
- note removed: "RECHECK ALL PINS"

Commit message: PCB_UPDATE
Parts:
- TP601, TP602: footprint TestPoint:TestPoint_Pad_D1.0mm -> Library:TP_0.5mm
Changed lines of the file:
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@@
 			)
 		)
-		(property "Footprint" "TestPoint:TestPoint_Pad_D1.0mm"
+		(property "Footprint" "Library:TP_0.5mm"
 			(at 34.29 83.82 0)
 			(effects
@@
 			)
 		)
-		(property "Footprint" "TestPoint:TestPoint_Pad_D1.0mm"
+		(property "Footprint" "Library:TP_0.5mm"
 			(at 54.61 83.82 0)
 			(effects
